File: r2/src/_usb-serial.kicad_sch (KiCad schematic)
At the start: 9 parts

Commit message: Set CP2102 IO voltage to 3.3V
Parts:
- removed R?: 0R, symbol Device:R_Small
Connections:
- net +1V8 is gone; now on net +3V3: C?.1, R?.1
- net +3V3: now reaches U?.5 (VIO)
Changed lines of the file:
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@@
     (stroke (width 0) (type solid) (color 0 0 0 0))
   )
-  (wire (pts (xy 161.29 70.485) (xy 161.29 72.39))
-    (stroke (width 0) (type solid) (color 0 0 0 0))
-  )
-  (wire (pts (xy 161.29 77.47) (xy 161.29 81.28))
+  (wire (pts (xy 161.29 70.485) (xy 161.29 81.28))
     (stroke (width 0) (type solid) (color 0 0 0 0))
   )
@@
     (pin "1")
   )
-  (symbol (lib_id "power:+1V8") (at 161.29 63.5 0) (unit 1)
+  (symbol (lib_id "power:+3V3") (at 161.29 63.5 0) (unit 1)
     (in_bom yes) (on_board yes)
     (property "Reference" "#PWR?" (id 0) (at 161.29 67.31 0)
       (effects (font (size 1.27 1.27)) hide)
     )
-    (property "Value" "+1V8" (id 1) (at 160.655 59.69 90)
-      (effects (font (size 1.27 1.27)) (justify left))
-    )
+    (property "Value" "+3V3" (id 1) (at 162.56 58.42 0))
     (property "Footprint" "" (id 2) (at 161.29 63.5 0)
       (effects (font (size 1.27 1.27)) hide)
@@
       (effects (font (size 1.27 1.27)) hide)
     )
-    (pin "1")
-    (pin "2")
-  )
-  (symbol (lib_id "Device:R_Small") (at 161.29 74.93 0) (unit 1)
-    (in_bom yes) (on_board yes)
-    (property "Reference" "R?" (id 0) (at 163.195 74.295 0)
-      (effects (font (size 1.27 1.27)) (justify left))
-    )
-    (property "Value" "0R" (id 1) (at 163.195 76.835 0)
-      (effects (font (size 1.27 1.27)) (justify left))
-    )
-    (property "Footprint" "" (id 2) (at 161.29 74.93 0)
-      (effects (font (size 1.27 1.27)) hide)
-    )
-    (property "Datasheet" "~" (id 3) (at 161.29 74.93 0)
-      (effects (font (size 1.27 1.27)) hide)
-    )
