File: r2/src/_modem.kicad_sch (KiCad schematic)
At the start: 36 parts, among them J1 , J2 , J3 , J4 , J4 JAE_SIM_Card_SF72S006, J5 , J6 , J7 , J8 , J9 , U8 Sierra_Wireless_RC7620, U9 ESD7004

Commit message: Annotate schematic, ERC pass
Parts:
- removed U9: ESD7004, Package_SON:USON-10_2.5x1.0mm_P0.5mm, symbol Power_Protection:TPD4E02B04DQA
- added U8: ESD7004, Package_SON:USON-10_2.5x1.0mm_P0.5mm, symbol Power_Protection:TPD4E02B04DQA
- gave numbers to parts that had none: 14
- renumbered C25 to C21, C26 to C22, C27 to C23, C28 to C24, C29 to C26, C30 to C28, D2 to D6, J4 to J13, R20 to R21, R21 to R22, R22 to R23, U8 to U7
Connections:
- net GND: now also U8.3 (G), U8.8 (G)
- net UIM_CLK_R: now also U8.4 (IO3); no longer C24.1, C26.1, C28.1, D6.2 (A2), J13.C1 (VCC), J13.C2 (RST), J13.C7 (I/O), J13.DSW, R21.1, R21.2, R22.1, R22.2, U7.26 (UIM1_VCC), U7.28 (UIM1_DATA), U7.29 (UIM1_RESET_N), U7.64 (UIM1_SIMA_DET)
- new net UIM_DATA: J13.C7 (I/O), R22.1, U7.28 (UIM1_DATA), U8.5 (IO4)
- new net UIM_RESET_N: J13.C2 (RST), U7.29 (UIM1_RESET_N), U8.2 (IO2)
- new net UIM_SIM_DET: D6.2 (A2), J13.DSW, R21.1, U7.64 (UIM1_SIMA_DET)
- new net UIM_VCC: C24.1, C26.1, C28.1, J13.C1 (VCC), R21.2, R22.2, U7.26 (UIM1_VCC), U8.1 (IO1)

Commit message: Footprint for modem
Parts:
- U7: footprint MODULE_WP7504 -> jeffmakes-footprints:Cellular_Modem-Sierra-Wireless-module-CF3-ringCD

Commit message: Most footprints assigned
Parts:
- C21, C25, C26, C27, C28: footprint (none) -> Capacitor_SMD:C_0603_1608Metric
- C22, C23, C24: footprint (none) -> Capacitor_SMD:C_0805_2012Metric
- J1, J2, J3, J4, J5, J6, J7, J8, J9, TP10, TP11, TP8, TP9: footprint (none) -> TestPoint:TestPoint_Pad_1.0x1.0mm
- J11: footprint (none) -> Connector_Coaxial:SMA_Amphenol_901-144_Vertical
- R21, R22, R23: footprint (none) -> Resistor_SMD:R_0603_1608Metric

Commit message: All footprints assigned
Parts:
- added D8, D9: 0402ESDA-MLP1, Diode_SMD:D_0402_1005Metric, symbol Device:D_TVS
Connections:
- net GND: now also D8.1 (A1), D9.1 (A1)
- net at J11.1 (In), R18.1: now also D8.2 (A2)
- net at J12.2, R19.1: now also D9.2 (A2)
Other:
- moved on the sheet: C19, C20, C21, C22, C23, C24, C26, C28, D6, J1, J11, J12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

Commit message: Change some footprints, change all testpoints to 1mm round.
Parts:
- J1, J2, J3, J4, J5, J6, J7, J8, J9, TP10, TP11, TP8, TP9: footprint TestPoint:TestPoint_Pad_1.0x1.0mm -> TestPoint:TestPoint_Pad_D1.0mm
- U8: footprint Package_SON:USON-10_2.5x1.0mm_P0.5mm -> jeffmakes-footprints:USON-10_2.5x1.0mm_P0.5mm
