File: r2/src/_rtc.kicad_sch (KiCad schematic)
At the start: 8 parts

Commit message: Annotate schematic, ERC pass
Parts:
- gave numbers to parts that had none: 8
Changed lines of the file:
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@@
+    (stroke (width 0) (type solid) (color 0 0 0 0))
+  )
+  (wire (pts (xy 106.68 71.12) (xy 106.68 72.39))
     (stroke (width 0) (type solid) (color 0 0 0 0))
   )
@@
     (stroke (width 0) (type solid) (color 0 0 0 0))
   )
-  (wire (pts (xy 191.77 99.06) (xy 198.12 99.06))
+  (wire (pts (xy 191.77 99.06) (xy 200.66 99.06))
     (stroke (width 0) (type solid) (color 0 0 0 0))
   )
@@
     (effects (font (size 1.27 1.27)) (justify right))
   )
-  (hierarchical_label "GLOBAL_EN" (shape output) (at 198.12 99.06 0)
+  (hierarchical_label "GLOBAL_EN" (shape output) (at 200.66 99.06 0)
     (effects (font (size 1.27 1.27)) (justify left))
   )
+  (symbol (lib_id "power:PWR_FLAG") (at 106.68 71.12 0) (unit 1)
+    (in_bom yes) (on_board yes)
+    (property "Reference" "#FLG0105" (id 0) (at 106.68 69.215 0)
+      (effects (font (size 1.27 1.27)) hide)
+    )
+    (property "Value" "PWR_FLAG" (id 1) (at 106.68 65.405 0))
+    (property "Footprint" "" (id 2) (at 106.68 71.12 0)
+      (effects (font (size 1.27 1.27)) hide)
+    )
+    (property "Datasheet" "~" (id 3) (at 106.68 71.12 0)
+      (effects (font (size 1.27 1.27)) hide)
+    )
+    (pin "1")
+  )
   (symbol (lib_id "power:+5V") (at 123.19 69.85 0) (unit 1)
     (in_bom yes) (on_board yes)
-    (property "Reference" "#PWR?" (id 0) (at 123.19 73.66 0)
+    (property "Reference" "#PWR0100" (id 0) (at 123.19 73.66 0)
       (effects (font (size 1.27 1.27)) hide)
     )
@@
   (symbol (lib_id "power:+5V") (at 185.42 76.2 0) (unit 1)
     (in_bom yes) (on_board yes)
-    (property "Reference" "#PWR?" (id 0) (at 185.42 80.01 0)
+    (property "Reference" "#PWR0103" (id 0) (at 185.42 80.01 0)
       (effects (font (size 1.27 1.27)) hide)
     )
@@
   (symbol (lib_id "power:GND") (at 93.98 81.28 0) (unit 1)
     (in_bom yes) (on_board yes)
-    (property "Reference" "#PWR?" (id 0) (at 93.98 87.63 0)
+    (property "Reference" "#PWR098" (id 0) (at 93.98 87.63 0)
       (effects (font (size 1.27 1.27)) hide)
     )
@@
   (symbol (lib_id "power:GND") (at 106.68 81.28 0) (unit 1)
     (in_bom yes) (on_board yes)
-    (property "Reference" "#PWR?" (id 0) (at 106.68 87.63 0)
+    (property "Reference" "#PWR099" (id 0) (at 106.68 87.63 0)
       (effects (font (size 1.27 1.27)) hide)
     )
@@
   (symbol (lib_id "power:GND") (at 123.19 107.95 0) (unit 1)
     (in_bom yes) (on_board yes)
-    (property "Reference" "#PWR?" (id 0) (at 123.19 114.3 0)
+    (property "Reference" "#PWR0101" (id 0) (at 123.19 114.3 0)
       (effects (font (size 1.27 1.27)) hide)
     )
@@
   (symbol (lib_id "power:GND") (at 128.27 81.28 0) (unit 1)
     (in_bom yes) (on_board yes)
-    (property "Reference" "#PWR?" (id 0) (at 128.27 87.63 0)
+    (property "Reference" "#PWR0102" (id 0) (at 128.27 87.63 0)
       (effects (font (size 1.27 1.27)) hide)
     )
@@
   (symbol (lib_id "power:GND") (at 185.42 107.95 0) (unit 1)
     (in_bom yes) (on_board yes)
-    (property "Reference" "#PWR?" (id 0) (at 185.42 114.3 0)
+    (property "Reference" "#PWR0104" (id 0) (at 185.42 114.3 0)
       (effects (font (size 1.27 1.27)) hide)
     )
@@
   (symbol (lib_id "Device:R_Small") (at 151.13 91.44 0) (mirror y) (unit 1)
     (in_bom yes) (on_board yes)
-    (property "Reference" "R?" (id 0) (at 153.67 90.17 0)
+    (property "Reference" "R29" (id 0) (at 153.67 90.17 0)
       (effects (font (size 1.27 1.27)) (justify right))
     )
@@
   (symbol (lib_id "Device:R_Small") (at 168.91 91.44 0) (mirror y) (unit 1)
     (in_bom yes) (on_board yes)
-    (property "Reference" "R?" (id 0) (at 171.45 90.17 0)
+    (property "Reference" "R30" (id 0) (at 171.45 90.17 0)
       (effects (font (size 1.27 1.27)) (justify right))
     )
@@
   (symbol (lib_id "Device:C_Small") (at 93.98 77.47 0) (unit 1)
     (in_bom yes) (on_board yes)
-    (property "Reference" "C?" (id 0) (at 96.52 76.2 0)
+    (property "Reference" "C34" (id 0) (at 96.52 76.2 0)
       (effects (font (size 1.27 1.27)) (justify left))
     )
@@
   (symbol (lib_id "Device:C_Small") (at 128.27 77.47 0) (unit 1)
     (in_bom yes) (on_board yes)
-    (property "Reference" "C?" (id 0) (at 130.81 76.2 0)
+    (property "Reference" "C35" (id 0) (at 130.81 76.2 0)
       (effects (font (size 1.27 1.27)) (justify left))
     )
@@
   (symbol (lib_id "Device:C_Small") (at 161.29 99.06 270) (unit 1)
     (in_bom yes) (on_board yes)
-    (property "Reference" "C?" (id 0) (at 161.29 102.87 90))
+    (property "Reference" "C36" (id 0) (at 161.29 102.87 90))
     (property "Value" "100nF" (id 1) (at 161.29 105.41 90))
     (property "Footprint" "" (id 2) (at 161.29 99.06 0)
@@
   (symbol (lib_id "Device:Battery_Cell") (at 106.68 78.74 0) (mirror y) (unit 1)
     (in_bom yes) (on_board yes)
-    (property "Reference" "BT?" (id 0) (at 110.49 76.2 0)
+    (property "Reference" "BT1" (id 0) (at 110.49 76.2 0)
       (effects (font (size 1.27 1.27)) (justify right))
     )
@@
   (symbol (lib_id "74xGxx:74LVC1G07") (at 185.42 99.06 0) (unit 1)
     (in_bom yes) (on_board yes)
-    (property "Reference" "U?" (id 0) (at 187.96 91.44 0))
+    (property "Reference" "U14" (id 0) (at 187.96 91.44 0))
     (property "Value" "74LVC1G07" (id 1) (at 191.77 93.98 0))
     (property "Footprint" "" (id 2) (at 185.42 99.06 0)
@@
   (symbol (lib_id "Timer_RTC:DS3231MZ") (at 123.19 96.52 0) (unit 1)
     (in_bom yes) (on_board yes)
-    (property "Reference" "U?" (id 0) (at 127 106.68 0))
+    (property "Reference" "U13" (id 0) (at 127 106.68 0))
     (property "Value" "DS3231MZ" (id 1) (at 130.81 109.22 0))
     (property "Footprint" "Package_SO:SOIC-8_3.9x4.9mm_P1.27mm" (id 2) (at 123.19 109.22 0)

Commit message: Most footprints assigned
Parts:
- C34, C35, C36: footprint (none) -> Capacitor_SMD:C_0603_1608Metric
- R29, R30: footprint (none) -> Resistor_SMD:R_0603_1608Metric
- U14: value 74LVC1G07 -> 74LVC1G07DCK; footprint (none) -> Package_TO_SOT_SMD:SOT-353_SC-70-5
Changed lines of the file:
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@@
       (effects (font (size 1.27 1.27)) (justify right))
     )
-    (property "Footprint" "" (id 2) (at 151.13 91.44 0)
+    (property "Footprint" "Resistor_SMD:R_0603_1608Metric" (id 2) (at 151.13 91.44 0)
       (effects (font (size 1.27 1.27)) hide)
     )
@@
       (effects (font (size 1.27 1.27)) (justify right))
     )
-    (property "Footprint" "" (id 2) (at 168.91 91.44 0)
+    (property "Footprint" "Resistor_SMD:R_0603_1608Metric" (id 2) (at 168.91 91.44 0)
       (effects (font (size 1.27 1.27)) hide)
     )
@@
       (effects (font (size 1.27 1.27)) (justify left))
     )
-    (property "Footprint" "" (id 2) (at 93.98 77.47 0)
+    (property "Footprint" "Capacitor_SMD:C_0603_1608Metric" (id 2) (at 93.98 77.47 0)
       (effects (font (size 1.27 1.27)) hide)
     )
@@
       (effects (font (size 1.27 1.27)) (justify left))
     )
-    (property "Footprint" "" (id 2) (at 128.27 77.47 0)
+    (property "Footprint" "Capacitor_SMD:C_0603_1608Metric" (id 2) (at 128.27 77.47 0)
       (effects (font (size 1.27 1.27)) hide)
     )
@@
     (property "Reference" "C36" (id 0) (at 161.29 102.87 90))
     (property "Value" "100nF" (id 1) (at 161.29 105.41 90))
-    (property "Footprint" "" (id 2) (at 161.29 99.06 0)
+    (property "Footprint" "Capacitor_SMD:C_0603_1608Metric" (id 2) (at 161.29 99.06 0)
       (effects (font (size 1.27 1.27)) hide)
     )
@@
   (symbol (lib_id "74xGxx:74LVC1G07") (at 185.42 99.06 0) (unit 1)
     (in_bom yes) (on_board yes)
-    (property "Reference" "U14" (id 0) (at 187.96 91.44 0))
-    (property "Value" "74LVC1G07" (id 1) (at 191.77 93.98 0))
-    (property "Footprint" "" (id 2) (at 185.42 99.06 0)
+    (property "Reference" "U14" (id 0) (at 189.23 91.44 0))
+    (property "Value" "74LVC1G07DCK" (id 1) (at 194.31 93.98 0))
+    (property "Footprint" "Package_TO_SOT_SMD:SOT-353_SC-70-5" (id 2) (at 185.42 99.06 0)
       (effects (font (size 1.27 1.27)) hide)
     )

Commit message: All footprints assigned
Parts:
- BT1: footprint (none) -> jeffmakes-footprints:Keystone-3000-CR1220-CR1216
Changed lines of the file:
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@@
       (effects (font (size 1.27 1.27)) (justify right))
     )
-    (property "Footprint" "" (id 2) (at 106.68 77.216 90)
+    (property "Footprint" "jeffmakes-footprints:Keystone-3000-CR1220-CR1216" (id 2) (at 106.68 77.216 90)
       (effects (font (size 1.27 1.27)) hide)
     )
