File: r2/src/_led_driver.kicad_sch (KiCad schematic)
At the start: 4 parts, among them J16 FH12-20S-0.5SVA, U17 PCA9685PW

Commit message: Most footprints assigned
Parts:
- C38: footprint (none) -> Capacitor_SMD:C_0603_1608Metric
- R33: footprint (none) -> Resistor_SMD:R_0603_1608Metric
Changed lines of the file:
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@@
       (effects (font (size 1.27 1.27)) (justify right))
     )
-    (property "Footprint" "" (id 2) (at 114.3 53.34 0)
+    (property "Footprint" "Resistor_SMD:R_0603_1608Metric" (id 2) (at 114.3 53.34 0)
       (effects (font (size 1.27 1.27)) hide)
     )
@@
       (effects (font (size 1.27 1.27)) (justify right))
     )
-    (property "Footprint" "" (id 2) (at 129.54 46.99 0)
+    (property "Footprint" "Capacitor_SMD:C_0603_1608Metric" (id 2) (at 129.54 46.99 0)
       (effects (font (size 1.27 1.27)) hide)
     )

Commit message: Change some footprints, change all testpoints to 1mm round.
Parts:
- J16: footprint jeffmakes-footprints:Hirose_FH12-20S-0.5SVA_1x20-1MP_P0.50mm_Vertical -> Connector_FFC-FPC:Hirose_FH12-20S-0.5SH_1x20-1MP_P0.50mm_Horizontal
Changed lines of the file:
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@@
       (effects (font (size 1.27 1.27)) (justify left))
     )
-    (property "Footprint" "jeffmakes-footprints:Hirose_FH12-20S-0.5SVA_1x20-1MP_P0.50mm_Vertical" (id 2) (at 189.23 72.39 0)
+    (property "Footprint" "Connector_FFC-FPC:Hirose_FH12-20S-0.5SH_1x20-1MP_P0.50mm_Horizontal" (id 2) (at 189.23 72.39 0)
       (effects (font (size 1.27 1.27)) hide)
     )

Commit message: Update schematic library symbols
Connections:
- net +3V3: no longer C38.1
- net GND: now also C38.1
Changed lines of the file:
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@@
   (junction (at 116.84 92.71) (diameter 1.016) (color 0 0 0 0))
   (junction (at 137.16 43.18) (diameter 1.016) (color 0 0 0 0))
-  (junction (at 137.16 50.8) (diameter 1.016) (color 0 0 0 0))
   (no_connect (at 154.94 74.93))
   (no_connect (at 154.94 82.55))
@@
     (stroke (width 0) (type solid) (color 0 0 0 0))
   )
-  (wire (pts (xy 129.54 50.8) (xy 137.16 50.8))
-    (stroke (width 0) (type solid) (color 0 0 0 0))
-  )
   (wire (pts (xy 137.16 41.91) (xy 137.16 43.18))
     (stroke (width 0) (type solid) (color 0 0 0 0))
   )
-  (wire (pts (xy 137.16 43.18) (xy 137.16 50.8))
-    (stroke (width 0) (type solid) (color 0 0 0 0))
-  )
-  (wire (pts (xy 137.16 50.8) (xy 137.16 52.07))
+  (wire (pts (xy 137.16 43.18) (xy 137.16 52.07))
     (stroke (width 0) (type solid) (color 0 0 0 0))
   )
@@
       (effects (font (size 1.27 1.27)) hide)
     )
+    (pin "1")
+  )
+  (symbol (lib_id "power:GND") (at 129.54 50.8 0) (unit 1)
+    (in_bom yes) (on_board yes)
+    (property "Reference" "#PWR0120" (id 0) (at 129.54 57.15 0)
+      (effects (font (size 1.27 1.27)) hide)
+    )
+    (property "Value" "GND" (id 1) (at 129.54 55.88 90))
+    (property "Footprint" "" (id 2) (at 129.54 50.8 0)
+      (effects (font (size 1.27 1.27)) hide)
+    )
+    (property "Datasheet" "" (id 3) (at 129.54 50.8 0)
+      (effects (font (size 1.27 1.27)) hide)
+    )

Commit message: Switch to LED connector with mmounting pad pins so we can solder the mounting pads to the more mechanically solid GND plane
Parts:
- removed J16: FH12-20S-0.5SVA, Connector_FFC-FPC:Hirose_FH12-20S-0.5SH_1x20-1MP_P0.50mm_Horizontal, symbol Connector_Generic:Conn_01x20
- added J16: FH12-20S-0.5SVA, Connector_FFC-FPC:Hirose_FH12-20S-0.5SH_1x20-1MP_P0.50mm_Horizontal, symbol Connector_Generic_MountingPin:Conn_01x20_MountingPin
Connections:
- net +3V3: now also J16.1 (Pin_1), J16.2 (Pin_2), J16.20 (Pin_20)
- net BCLK: now also J16.15 (Pin_15)
- net FSYNC: now also J16.16 (Pin_16)
- net GND: now also J16.3 (Pin_3), J16.4 (Pin_4), J16.MP (MountPin)
- net LED1_B: now also J16.7 (Pin_7)
- net LED1_G: now also J16.6 (Pin_6)
- net LED1_R: now also J16.5 (Pin_5)
- net LED2_B: now also J16.10 (Pin_10)
- net LED2_G: now also J16.9 (Pin_9)
- net LED2_R: now also J16.8 (Pin_8)
- net LED3_B: now also J16.13 (Pin_13)
- net LED3_G: now also J16.12 (Pin_12)
- net LED3_R: now also J16.11 (Pin_11)
- net SCL: now also J16.18 (Pin_18)
- net SDA: now also J16.17 (Pin_17)
- net SDOUT: now also J16.14 (Pin_14)
- net SHDNZ: now also J16.19 (Pin_19)
Changed lines of the file:
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@@
+    (pin "1")
+  )
+  (symbol (lib_id "power:GND") (at 189.23 102.87 0) (unit 1)
+    (in_bom yes) (on_board yes)
+    (property "Reference" "#PWR0122" (id 0) (at 189.23 109.22 0)
+      (effects (font (size 1.27 1.27)) hide)
+    )
+    (property "Value" "GND" (id 1) (at 190.5 107.95 0))
+    (property "Footprint" "" (id 2) (at 189.23 102.87 0)
+      (effects (font (size 1.27 1.27)) hide)
+    )
+    (property "Datasheet" "" (id 3) (at 189.23 102.87 0)
+      (effects (font (size 1.27 1.27)) hide)
+    )
     (pin "1")
   )
@@
     (pin "2")
   )
-  (symbol (lib_id "Connector_Generic:Conn_01x20") (at 189.23 72.39 0) (unit 1)
+  (symbol (lib_id "Connector_Generic_MountingPin:Conn_01x20_MountingPin") (at 189.23 72.39 0) (unit 1)
     (in_bom yes) (on_board yes)
-    (property "Reference" "J16" (id 0) (at 192.405 71.755 0)
+    (property "Reference" "J16" (id 0) (at 191.77 75.0569 0)
       (effects (font (size 1.27 1.27)) (justify left))
     )
-    (property "Value" "FH12-20S-0.5SVA" (id 1) (at 192.405 74.295 0)
+    (property "Value" "FH12-20S-0.5SVA" (id 1) (at 191.77 77.5969 0)
       (effects (font (size 1.27 1.27)) (justify left))
     )
@@
     (pin "8")
     (pin "9")
+    (pin "MP")
   )
   (symbol (lib_id "Driver_LED:PCA9685PW") (at 137.16 77.47 0) (unit 1)

Commit message: Add 5V connection to LED connector pin 20. Switch to using 5V rail to power leds to reduce noise
Parts:
- J16: value FH12-20S-0.5SVA -> FH12A-20S-0.5SH
Connections:
- net +3V3: no longer J16.20 (Pin_20)
- new net +5V: J16.20 (Pin_20)
Changed lines of the file:
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@@
-    (stroke (width 0) (type solid) (color 0 0 0 0))
-  )
-  (wire (pts (xy 173.99 97.79) (xy 184.15 97.79))
     (stroke (width 0) (type solid) (color 0 0 0 0))
   )
@@
   )
   (wire (pts (xy 175.26 57.15) (xy 184.15 57.15))
+    (stroke (width 0) (type solid) (color 0 0 0 0))
+  )
+  (wire (pts (xy 175.26 97.79) (xy 184.15 97.79))
     (stroke (width 0) (type solid) (color 0 0 0 0))
   )
@@
     (effects (font (size 1.27 1.27)) (justify left bottom))
   )
-  (label "+3V3" (at 173.99 97.79 0)
-    (effects (font (size 1.27 1.27)) (justify left bottom))
-  )
-  (label "+3V3" (at 175.26 49.53 0)
-    (effects (font (size 1.27 1.27)) (justify left bottom))
-  )
-  (label "+3V3" (at 175.26 52.07 0)
-    (effects (font (size 1.27 1.27)) (justify left bottom))
-  )
-  (label "GND" (at 175.26 54.61 0)
-    (effects (font (size 1.27 1.27)) (justify left bottom))
-  )
-  (label "GND" (at 175.26 57.15 0)
-    (effects (font (size 1.27 1.27)) (justify left bottom))
-  )
   (label "LED1_R" (at 175.26 59.69 0)
     (effects (font (size 1.27 1.27)) (justify left bottom))
@@
     (pin "1")
   )
+  (symbol (lib_id "power:+3V3") (at 175.26 49.53 90) (unit 1)
+    (in_bom yes) (on_board yes)
+    (property "Reference" "#PWR?" (id 0) (at 179.07 49.53 0)
+      (effects (font (size 1.27 1.27)) hide)
+    )
+    (property "Value" "+3V3" (id 1) (at 168.91 49.53 90))
+    (property "Footprint" "" (id 2) (at 175.26 49.53 0)
+      (effects (font (size 1.27 1.27)) hide)
+    )
+    (property "Datasheet" "" (id 3) (at 175.26 49.53 0)
+      (effects (font (size 1.27 1.27)) hide)
+    )
+    (pin "1")
+  )
+  (symbol (lib_id "power:+3V3") (at 175.26 52.07 90) (unit 1)
+    (in_bom yes) (on_board yes)
+    (property "Reference" "#PWR?" (id 0) (at 179.07 52.07 0)
+      (effects (font (size 1.27 1.27)) hide)
+    )
+    (property "Value" "+3V3" (id 1) (at 168.91 52.07 90))
+    (property "Footprint" "" (id 2) (at 175.26 52.07 0)
+      (effects (font (size 1.27 1.27)) hide)
+    )
+    (property "Datasheet" "" (id 3) (at 175.26 52.07 0)
+      (effects (font (size 1.27 1.27)) hide)
+    )
+    (pin "1")
+  )
+  (symbol (lib_id "power:+5V") (at 175.26 97.79 90) (unit 1)
+    (in_bom yes) (on_board yes)
+    (property "Reference" "#PWR?" (id 0) (at 179.07 97.79 0)
+      (effects (font (size 1.27 1.27)) hide)
+    )
+    (property "Value" "+5V" (id 1) (at 171.45 98.4249 90)
+      (effects (font (size 1.27 1.27)) (justify left))
+    )
+    (property "Footprint" "" (id 2) (at 175.26 97.79 0)
+      (effects (font (size 1.27 1.27)) hide)
+    )
+    (property "Datasheet" "" (id 3) (at 175.26 97.79 0)
+      (effects (font (size 1.27 1.27)) hide)
+    )
+    (pin "1")
+  )
   (symbol (lib_id "power:GND") (at 111.76 64.77 270) (unit 1)
     (in_bom yes) (on_board yes)
@@
     (pin "1")
   )
+  (symbol (lib_id "power:GND") (at 175.26 54.61 270) (unit 1)
+    (in_bom yes) (on_board yes)
+    (property "Reference" "#PWR?" (id 0) (at 168.91 54.61 0)
+      (effects (font (size 1.27 1.27)) hide)
+    )
+    (property "Value" "GND" (id 1) (at 171.45 55.2449 90)
+      (effects (font (size 1.27 1.27)) (justify right))
+    )
+    (property "Footprint" "" (id 2) (at 175.26 54.61 0)
+      (effects (font (size 1.27 1.27)) hide)
+    )
+    (property "Datasheet" "" (id 3) (at 175.26 54.61 0)
+      (effects (font (size 1.27 1.27)) hide)
+    )
+    (pin "1")
+  )
+  (symbol (lib_id "power:GND") (at 175.26 57.15 270) (unit 1)
+    (in_bom yes) (on_board yes)
+    (property "Reference" "#PWR?" (id 0) (at 168.91 57.15 0)
+      (effects (font (size 1.27 1.27)) hide)
+    )
+    (property "Value" "GND" (id 1) (at 171.45 57.7849 90)
+      (effects (font (size 1.27 1.27)) (justify right))
+    )
+    (property "Footprint" "" (id 2) (at 175.26 57.15 0)
+      (effects (font (size 1.27 1.27)) hide)
+    )
+    (property "Datasheet" "" (id 3) (at 175.26 57.15 0)
+      (effects (font (size 1.27 1.27)) hide)
+    )
+    (pin "1")
+  )
   (symbol (lib_id "power:GND") (at 189.23 102.87 0) (unit 1)
     (in_bom yes) (on_board yes)
@@
       (effects (font (size 1.27 1.27)) (justify left))
     )
-    (property "Value" "FH12-20S-0.5SVA" (id 1) (at 191.77 77.5969 0)
+    (property "Value" "FH12A-20S-0.5SH" (id 1) (at 191.77 77.5969 0)
       (effects (font (size 1.27 1.27)) (justify left))
     )
