File: r3/src/safeproject-main-r3.kicad_sch (KiCad schematic)
At the start: 28 parts, among them T1 , T3 , T4 , T5 , T6 , T7 , U1 74LVC1G07DCK

Commit message: Add 1.8V test point.
Parts:
- added T2: (no value), TestPoint:TestPoint_Pad_D1.0mm, symbol Connector:TestPoint
Connections:
- net +1V8: now also T2.1
Changed lines of the file:
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@@
     (stroke (width 0) (type solid) (color 0 0 0 0))
   )
-  (wire (pts (xy 173.99 170.18) (xy 179.07 170.18))
+  (wire (pts (xy 166.37 185.42) (xy 176.53 185.42))
     (stroke (width 0) (type solid) (color 0 0 0 0))
   )
-  (wire (pts (xy 173.99 180.34) (xy 176.53 180.34))
+  (wire (pts (xy 173.99 170.18) (xy 179.07 170.18))
     (stroke (width 0) (type solid) (color 0 0 0 0))
   )
-  (wire (pts (xy 173.99 185.42) (xy 176.53 185.42))
+  (wire (pts (xy 173.99 180.34) (xy 176.53 180.34))
     (stroke (width 0) (type solid) (color 0 0 0 0))
   )
@@
     (effects (font (size 1.27 1.27)) (justify left bottom))
   )
+  (label "+1V8" (at 167.005 185.42 0)
+    (effects (font (size 1.27 1.27)) (justify left bottom))
+  )
   (label "TX_ON" (at 264.16 104.14 180)
     (effects (font (size 1.27 1.27)) (justify right bottom))
@@
     (pin "1")
   )
-  (symbol (lib_id "power:+1V8") (at 173.99 185.42 90) (unit 1)
-    (in_bom yes) (on_board yes)
-    (property "Reference" "#PWR035" (id 0) (at 177.8 185.42 0)
-      (effects (font (size 1.27 1.27)) hide)
-    )
-    (property "Value" "+1V8" (id 1) (at 170.18 186.055 90)
-      (effects (font (size 1.27 1.27)) (justify left))
-    )
-    (property "Footprint" "" (id 2) (at 173.99 185.42 0)
-      (effects (font (size 1.27 1.27)) hide)
-    )
-    (property "Datasheet" "" (id 3) (at 173.99 185.42 0)
-      (effects (font (size 1.27 1.27)) hide)
-    )
-    (pin "1")
-  )
   (symbol (lib_id "power:+5V") (at 245.11 170.18 270) (unit 1)
     (in_bom yes) (on_board yes)
@@
     (pin "1")
   )
+  (symbol (lib_id "Connector:TestPoint") (at 166.37 185.42 90) (unit 1)
+    (in_bom yes) (on_board yes)
+    (property "Reference" "T2" (id 0) (at 161.29 185.42 90)
+      (effects (font (size 1.27 1.27)) (justify left))
+    )
+    (property "Value" " " (id 1) (at 161.29 186.69 90)
+      (effects (font (size 1.27 1.27)) (justify left))
+    )
+    (property "Footprint" "TestPoint:TestPoint_Pad_D1.0mm" (id 2) (at 166.37 180.34 0)
+      (effects (font (size 1.27 1.27)) hide)
+    )
+    (property "Datasheet" "~" (id 3) (at 166.37 180.34 0)
+      (effects (font (size 1.27 1.27)) hide)
+    )
+    (pin "1")
+  )
   (symbol (lib_id "Connector:TestPoint") (at 179.07 116.84 90) (unit 1)
     (in_bom yes) (on_board yes)
@@
   (symbol (lib_id "power:GND") (at 129.54 226.06 0) (unit 1)
     (in_bom yes) (on_board yes)
-    (property "Reference" "#PWR?" (id 0) (at 129.54 232.41 0)
+    (property "Reference" "#PWR0144" (id 0) (at 129.54 232.41 0)
       (effects (font (size 1.27 1.27)) hide)
     )
@@
   (symbol (lib_id "power:GND") (at 129.54 237.49 0) (unit 1)
     (in_bom yes) (on_board yes)
-    (property "Reference" "#PWR?" (id 0) (at 129.54 243.84 0)
+    (property "Reference" "#PWR0145" (id 0) (at 129.54 243.84 0)
       (effects (font (size 1.27 1.27)) hide)
     )
@@
   (symbol (lib_id "power:GND") (at 129.54 248.92 0) (unit 1)
     (in_bom yes) (on_board yes)
-    (property "Reference" "#PWR?" (id 0) (at 129.54 255.27 0)
+    (property "Reference" "#PWR0146" (id 0) (at 129.54 255.27 0)
       (effects (font (size 1.27 1.27)) hide)
     )
@@
   (symbol (lib_id "power:GND") (at 129.54 260.35 0) (unit 1)
     (in_bom yes) (on_board yes)
-    (property "Reference" "#PWR?" (id 0) (at 129.54 266.7 0)
+    (property "Reference" "#PWR0147" (id 0) (at 129.54 266.7 0)
       (effects (font (size 1.27 1.27)) hide)
     )
@@
       (reference "#PWR034") (unit 1) (value "+3V3") (footprint "")
     )
-    (path "/2d127711-d4f8-402a-a37e-05e2a2a8c854"
-      (reference "#PWR035") (unit 1) (value "+1V8") (footprint "")
-    )
     (path "/0e2c286d-da78-422c-a039-4f51a88a5b9a"
       (reference "#PWR036") (unit 1) (value "GND") (footprint "")
@@
     )
     (path "/0dd43c1f-99c9-4210-8986-6e3fd0c15cbd"
-      (reference "#PWR?") (unit 1) (value "GND") (footprint "")
+      (reference "#PWR0144") (unit 1) (value "GND") (footprint "")
+    )
+    (path "/cc50959c-924e-48f9-8d70-198206a6dabf"
+      (reference "#PWR0145") (unit 1) (value "GND") (footprint "")
     )
     (path "/a59e8e71-9992-4fe8-b136-c31752c9bccc"
-      (reference "#PWR?") (unit 1) (value "GND") (footprint "")
+      (reference "#PWR0146") (unit 1) (value "GND") (footprint "")
     )
     (path "/be2d00d6-ead2-4e5f-8896-24a88c32d929"
-      (reference "#PWR?") (unit 1) (value "GND") (footprint "")
-    )
-    (path "/cc50959c-924e-48f9-8d70-198206a6dabf"
-      (reference "#PWR?") (unit 1) (value "GND") (footprint "")
+      (reference "#PWR0147") (unit 1) (value "GND") (footprint "")
     )
     (path "/41dcda57-f03b-4254-a26d-4b483d171c17/80bf2495-1999-475f-8d3c-7c216f4c07f0"
@@
       (reference "T1") (unit 1) (value " ") (footprint "TestPoint:TestPoint_Pad_D1.0mm")
     )
+    (path "/7029dc71-5612-47e1-a070-8bab3ee33f42"
+      (reference "T2") (unit 1) (value " ") (footprint "TestPoint:TestPoint_Pad_D1.0mm")
+    )
     (path "/a28dff5b-6aea-45e3-a447-6ff0232d5c28"
       (reference "T3") (unit 1) (value " ") (footprint "TestPoint:TestPoint_Pad_D1.0mm")
@@
       (reference "T11") (unit 1) (value " ") (footprint "TestPoint:TestPoint_Pad_D1.0mm")
     )
+    (path "/e93db74d-0429-4e7f-b256-c16b4c3a83e7/10568141-439e-4479-867b-c8b4e8c1d987"
+      (reference "T12") (unit 1) (value " ") (footprint "TestPoint:TestPoint_Pad_D1.0mm")
+    )
+    (path "/e93db74d-0429-4e7f-b256-c16b4c3a83e7/13eaa826-bbb5-4091-ae72-ba242e352a0f"
+      (reference "T13") (unit 1) (value " ") (footprint "TestPoint:TestPoint_Pad_D1.0mm")
+    )
     (path "/0d301e3a-5e66-4f12-a600-824f82e690fc"

Commit message: Test points routed
Parts:
- added T14, T15, T16: (no value), TestPoint:TestPoint_Pad_D1.0mm, symbol Connector:TestPoint
Connections:
- net GLOBAL_EN_o: now also T16.1
- net SCL: now also T15.1
- net SDA: now also T14.1
Changed lines of the file:
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@@
   (paper "A3")
   (junction (at 147.32 142.24) (diameter 1.016) (color 0 0 0 0))
+  (junction (at 163.195 144.78) (diameter 1.016) (color 0 0 0 0))
+  (junction (at 165.735 142.24) (diameter 1.016) (color 0 0 0 0))
   (junction (at 176.53 180.34) (diameter 1.016) (color 0 0 0 0))
   (junction (at 176.53 185.42) (diameter 1.016) (color 0 0 0 0))
@@
     (stroke (width 0) (type solid) (color 0 0 0 0))
   )
-  (wire (pts (xy 153.67 142.24) (xy 179.07 142.24))
+  (wire (pts (xy 153.67 142.24) (xy 165.735 142.24))
     (stroke (width 0) (type solid) (color 0 0 0 0))
   )
-  (wire (pts (xy 153.67 144.78) (xy 179.07 144.78))
+  (wire (pts (xy 153.67 144.78) (xy 163.195 144.78))
     (stroke (width 0) (type solid) (color 0 0 0 0))
   )
@@
     (stroke (width 0) (type solid) (color 0 0 0 0))
   )
+  (wire (pts (xy 163.195 144.78) (xy 163.195 146.685))
+    (stroke (width 0) (type solid) (color 0 0 0 0))
+  )
+  (wire (pts (xy 163.195 144.78) (xy 179.07 144.78))
+    (stroke (width 0) (type solid) (color 0 0 0 0))
+  )
+  (wire (pts (xy 165.735 142.24) (xy 165.735 146.685))
+    (stroke (width 0) (type solid) (color 0 0 0 0))
+  )
+  (wire (pts (xy 165.735 142.24) (xy 179.07 142.24))
+    (stroke (width 0) (type solid) (color 0 0 0 0))
+  )
   (wire (pts (xy 166.37 185.42) (xy 176.53 185.42))
     (stroke (width 0) (type solid) (color 0 0 0 0))
@@
     (pin "1")
   )
+  (symbol (lib_id "Connector:TestPoint") (at 163.195 146.685 180) (unit 1)
+    (in_bom yes) (on_board yes)
+    (property "Reference" "T14" (id 0) (at 163.195 151.765 90)
+      (effects (font (size 1.27 1.27)) (justify left))
+    )
+    (property "Value" " " (id 1) (at 164.465 151.765 90)
+      (effects (font (size 1.27 1.27)) (justify left))
+    )
+    (property "Footprint" "TestPoint:TestPoint_Pad_D1.0mm" (id 2) (at 158.115 146.685 0)
+      (effects (font (size 1.27 1.27)) hide)
+    )
+    (property "Datasheet" "~" (id 3) (at 158.115 146.685 0)
+      (effects (font (size 1.27 1.27)) hide)
+    )
+    (pin "1")
+  )
+  (symbol (lib_id "Connector:TestPoint") (at 165.735 146.685 180) (unit 1)
+    (in_bom yes) (on_board yes)
+    (property "Reference" "T15" (id 0) (at 165.735 151.765 90)
+      (effects (font (size 1.27 1.27)) (justify left))
+    )
+    (property "Value" " " (id 1) (at 167.005 151.765 90)
+      (effects (font (size 1.27 1.27)) (justify left))
+    )
+    (property "Footprint" "TestPoint:TestPoint_Pad_D1.0mm" (id 2) (at 160.655 146.685 0)
+      (effects (font (size 1.27 1.27)) hide)
+    )
+    (property "Datasheet" "~" (id 3) (at 160.655 146.685 0)
+      (effects (font (size 1.27 1.27)) hide)
+    )
+    (pin "1")
+  )
   (symbol (lib_id "Connector:TestPoint") (at 166.37 185.42 90) (unit 1)
     (in_bom yes) (on_board yes)
@@
     (pin "1")
   )
+  (symbol (lib_id "Connector:TestPoint") (at 264.16 198.12 270) (unit 1)
+    (in_bom yes) (on_board yes)
+    (property "Reference" "T16" (id 0) (at 269.24 198.12 90)
+      (effects (font (size 1.27 1.27)) (justify left))
+    )
+    (property "Value" " " (id 1) (at 269.24 196.85 90)
+      (effects (font (size 1.27 1.27)) (justify left))
+    )
+    (property "Footprint" "TestPoint:TestPoint_Pad_D1.0mm" (id 2) (at 264.16 203.2 0)
+      (effects (font (size 1.27 1.27)) hide)
+    )
+    (property "Datasheet" "~" (id 3) (at 264.16 203.2 0)
+      (effects (font (size 1.27 1.27)) hide)
+    )
+    (pin "1")
+  )
   (symbol (lib_id "power:GND") (at 52.07 81.28 270) (unit 1)
     (in_bom yes) (on_board yes)
@@
       (reference "T13") (unit 1) (value " ") (footprint "TestPoint:TestPoint_Pad_D1.0mm")
     )
+    (path "/fcb49e07-a2a2-4397-af2b-8defe95e017e"
+      (reference "T14") (unit 1) (value " ") (footprint "TestPoint:TestPoint_Pad_D1.0mm")
+    )
+    (path "/2a0442cb-5411-48c8-925c-f59398e20545"
+      (reference "T15") (unit 1) (value " ") (footprint "TestPoint:TestPoint_Pad_D1.0mm")
+    )
+    (path "/9ccdc2ea-4360-4b47-aed5-c03dd29ae59e"
+      (reference "T16") (unit 1) (value " ") (footprint "TestPoint:TestPoint_Pad_D1.0mm")
+    )
     (path "/0d301e3a-5e66-4f12-a600-824f82e690fc"
