File: r3/src/safeproject-main-r3.kicad_sch (KiCad schematic)
At the start: 32 parts, among them T1 , T14 , T15 , T16 , T2 , T3 , T4 , T5 , T6 , T7 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

Commit message: Create a variant of the pi without holes, so they don't interfere with the Wurth spacer holes. Fix the mounting holes to create bare FR4 regions as in r2. New variant of the spacers with connectable pads. Spacers are connected to GND plane
Parts:
- Module1: footprint Raspberry_Pi_CM4:Raspberry-Pi-4-Compute-Module -> jeffmakes-footprints:Raspberry-Pi-4-Compute-Module-no-holes
Changed lines of the file:
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@@
     )
   )
-  (symbol (lib_id "Mechanical:MountingHole_Pad") (at 129.54 223.52 0) (unit 1)
+  (symbol (lib_name "Mechanical:MountingHole_Pad_1") (lib_id "Mechanical:MountingHole_Pad") (at 129.54 223.52 0) (unit 1)
     (in_bom yes) (on_board yes)
     (property "Reference" "SP1" (id 0) (at 133.35 222.8849 0)
@@
     (property "Reference" "Module1" (id 0) (at 83.185 204.0444 0))
     (property "Value" "ComputeModule4-CM4" (id 1) (at 83.185 206.3431 0))
-    (property "Footprint" "Raspberry_Pi_CM4:Raspberry-Pi-4-Compute-Module" (id 2) (at 85.09 161.29 0)
+    (property "Footprint" "jeffmakes-footprints:Raspberry-Pi-4-Compute-Module-no-holes" (id 2) (at 85.09 161.29 0)
       (effects (font (size 1.27 1.27)) hide)
     )
@@
     (property "Reference" "Module1" (id 0) (at 210.82 203.4094 0))
     (property "Value" "ComputeModule4-CM4" (id 1) (at 210.82 205.7081 0))
-    (property "Footprint" "Raspberry_Pi_CM4:Raspberry-Pi-4-Compute-Module" (id 2) (at 354.33 156.21 0)
+    (property "Footprint" "jeffmakes-footprints:Raspberry-Pi-4-Compute-Module-no-holes" (id 2) (at 354.33 156.21 0)
       (effects (font (size 1.27 1.27)) hide)
     )
@@
     )
     (path "/983969c3-711c-41cf-b33f-8b265354541d"
-      (reference "Module1") (unit 1) (value "ComputeModule4-CM4") (footprint "Raspberry_Pi_CM4:Raspberry-Pi-4-Compute-Module")
+      (reference "Module1") (unit 1) (value "ComputeModule4-CM4") (footprint "jeffmakes-footprints:Raspberry-Pi-4-Compute-Module-no-holes")
     )
     (path "/2e5d8954-dabb-4a70-9f83-592efa0a244f"
-      (reference "Module1") (unit 2) (value "ComputeModule4-CM4") (footprint "Raspberry_Pi_CM4:Raspberry-Pi-4-Compute-Module")
+      (reference "Module1") (unit 2) (value "ComputeModule4-CM4") (footprint "jeffmakes-footprints:Raspberry-Pi-4-Compute-Module-no-holes")
     )
     (path "/e93db74d-0429-4e7f-b256-c16b4c3a83e7/8b1ef4d6-8826-499c-8a98-a982520e62d5"
