File: r3/src/_sdcard.kicad_sch (KiCad schematic)
At the start: 6 parts, among them J14 Micro_SD_Card_Det_JAE_ST11, U10 ESD7004, U11 ESD7004

Commit message: Change to new 5-pin variant of the protection diode network symbol
Parts:
- U10, U11: footprint jeffmakes-footprints:USON-10_2.5x1.0mm_P0.5mm -> Package_SON:USON-10_2.5x1.0mm_P0.5mm; symbol Power_Protection:TPD4E02B04DQA -> j_Power_Protection:ESD7004
Connections:
- net GND: no longer U10.8 (G), U11.8 (G)
Changed lines of the file:
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@@
     (pin "2")
   )
-  (symbol (lib_id "Power_Protection:TPD4E02B04DQA") (at 118.11 123.19 0) (unit 1)
+  (symbol (lib_id "j_Power_Protection:ESD7004") (at 118.11 123.19 0) (unit 1)
     (in_bom yes) (on_board yes)
     (property "Reference" "U10" (id 0) (at 120.65 128.27 0)
@@
       (effects (font (size 1.27 1.27)) (justify left))
     )
-    (property "Footprint" "jeffmakes-footprints:USON-10_2.5x1.0mm_P0.5mm" (id 2) (at 125.73 123.19 0)
+    (property "Footprint" "Package_SON:USON-10_2.5x1.0mm_P0.5mm" (id 2) (at 125.73 123.19 0)
       (effects (font (size 1.27 1.27)) (justify left) hide)
     )
@@
     (pin "3")
     (pin "1")
-    (pin "10")
     (pin "2")
     (pin "4")
     (pin "5")
-    (pin "6")
-    (pin "7")
-    (pin "8")
-    (pin "9")
   )
-  (symbol (lib_id "Power_Protection:TPD4E02B04DQA") (at 135.89 123.19 0) (unit 1)
+  (symbol (lib_id "j_Power_Protection:ESD7004") (at 135.89 123.19 0) (unit 1)
     (in_bom yes) (on_board yes)
     (property "Reference" "U11" (id 0) (at 138.43 128.27 0)
@@
       (effects (font (size 1.27 1.27)) (justify left))
     )
-    (property "Footprint" "jeffmakes-footprints:USON-10_2.5x1.0mm_P0.5mm" (id 2) (at 143.51 123.19 0)
+    (property "Footprint" "Package_SON:USON-10_2.5x1.0mm_P0.5mm" (id 2) (at 143.51 123.19 0)
       (effects (font (size 1.27 1.27)) (justify left) hide)
     )
@@
     (pin "3")
     (pin "1")
-    (pin "10")
     (pin "2")
     (pin "4")
     (pin "5")
-    (pin "6")
-    (pin "7")
-    (pin "8")
-    (pin "9")
   )
   (symbol (lib_id "j_Connector:Micro_SD_Card_Det_JAE_ST11") (at 182.88 102.87 0) (unit 1)

Commit message: Change all diode protection networks to a 5-pin variant to prevent DRC errors due to missing pads
Parts:
- U10, U11: footprint Package_SON:USON-10_2.5x1.0mm_P0.5mm -> jeffmakes-footprints:USON-10_2.5x1.0mm_P0.5mm
Changed lines of the file:
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@@
       (effects (font (size 1.27 1.27)) (justify left))
     )
-    (property "Footprint" "Package_SON:USON-10_2.5x1.0mm_P0.5mm" (id 2) (at 125.73 123.19 0)
+    (property "Footprint" "jeffmakes-footprints:USON-10_2.5x1.0mm_P0.5mm" (id 2) (at 125.73 123.19 0)
       (effects (font (size 1.27 1.27)) (justify left) hide)
     )
@@
       (effects (font (size 1.27 1.27)) (justify left))
     )
-    (property "Footprint" "Package_SON:USON-10_2.5x1.0mm_P0.5mm" (id 2) (at 143.51 123.19 0)
+    (property "Footprint" "jeffmakes-footprints:USON-10_2.5x1.0mm_P0.5mm" (id 2) (at 143.51 123.19 0)
       (effects (font (size 1.27 1.27)) (justify left) hide)
     )
