File: r3/src/_usb_otg.kicad_sch (KiCad schematic)
At the start: 7 parts, among them J15 10118194, Q4 NX3008NBKW, U15 FSUSB42MX, U16 ESD7004

Commit message: Change to new 5-pin variant of the protection diode network symbol
Parts:
- U16: footprint jeffmakes-footprints:USON-10_2.5x1.0mm_P0.5mm -> Package_SON:USON-10_2.5x1.0mm_P0.5mm; symbol Power_Protection:TPD4E02B04DQA -> j_Power_Protection:ESD7004
Connections:
- net GND: no longer U16.8 (G)
Changed lines of the file:
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@@
     (pin "3")
   )
-  (symbol (lib_id "Power_Protection:TPD4E02B04DQA") (at 172.72 120.65 0) (unit 1)
+  (symbol (lib_id "j_Power_Protection:ESD7004") (at 172.72 120.65 0) (unit 1)
     (in_bom yes) (on_board yes)
     (property "Reference" "U16" (id 0) (at 180.34 118.11 0)
@@
       (effects (font (size 1.27 1.27)) (justify left))
     )
-    (property "Footprint" "jeffmakes-footprints:USON-10_2.5x1.0mm_P0.5mm" (id 2) (at 180.34 120.65 0)
+    (property "Footprint" "Package_SON:USON-10_2.5x1.0mm_P0.5mm" (id 2) (at 180.34 120.65 0)
       (effects (font (size 1.27 1.27)) (justify left) hide)
     )
@@
     (pin "3")
     (pin "1")
-    (pin "10")
     (pin "2")
     (pin "4")
     (pin "5")
-    (pin "6")
-    (pin "7")
-    (pin "8")
-    (pin "9")
   )
   (symbol (lib_id "Connector:USB_B_Micro") (at 207.01 106.68 0) (mirror y) (unit 1)

Commit message: Change all diode protection networks to a 5-pin variant to prevent DRC errors due to missing pads
Parts:
- U16: footprint Package_SON:USON-10_2.5x1.0mm_P0.5mm -> jeffmakes-footprints:USON-10_2.5x1.0mm_P0.5mm
Changed lines of the file:
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@@
       (effects (font (size 1.27 1.27)) (justify left))
     )
-    (property "Footprint" "Package_SON:USON-10_2.5x1.0mm_P0.5mm" (id 2) (at 180.34 120.65 0)
+    (property "Footprint" "jeffmakes-footprints:USON-10_2.5x1.0mm_P0.5mm" (id 2) (at 180.34 120.65 0)
       (effects (font (size 1.27 1.27)) (justify left) hide)
     )
