File: r4/src/_modem.kicad_sch (KiCad schematic)
At the start: 50 parts

Commit message: Add netclass definitions and assign nets. Define DRC rules to each class. Resize all vias and nets (with a few exceptions for very wide power tracks) to follow the netclass rules. Increase area for GNDA domain. Re-route SIM data bus around edge of GNDA domain
Parts:
- C19, C20: renamed from ?; value (none) -> DNP; footprint (none) -> Capacitor_SMD:C_0402_1005Metric
- C21: renamed from ?; value (none) -> 15pF; footprint (none) -> Capacitor_SMD:C_0603_1608Metric
- C22, C23: renamed from ?; value (none) -> 47uF; footprint (none) -> Capacitor_SMD:C_0805_2012Metric
- C24: renamed from ?; value (none) -> DNP 4.7uF; footprint (none) -> Capacitor_SMD:C_0805_2012Metric
- C26: renamed from ?; value (none) -> 100nF; footprint (none) -> Capacitor_SMD:C_0603_1608Metric
- C28: renamed from ?; value (none) -> 1nF; footprint (none) -> Capacitor_SMD:C_0603_1608Metric
- D3: renamed from ?; value (none) -> LO R976-PS-1; footprint (none) -> jeffmakes-footprints:CHIPLED-0805
- D6, D9: renamed from ?; value (none) -> 0402ESDA-MLP1; footprint (none) -> Diode_SMD:D_0402_1005Metric
- J1, J2, J3, J4, J5, J6, J7, J8, J9, T10, T11, T8, T9: renamed from ?; value (none) -> (none); footprint (none) -> TestPoint:TestPoint_Pad_D1.0mm
- J11: renamed from ?; value (none) -> SMA; footprint (none) -> Connector_Coaxial:SMA_Amphenol_132134-10_Vertical
- J12: renamed from ?; value (none) -> U_FL-R-SMT-1_10_; footprint (none) -> Connector_Coaxial:U.FL_Hirose_U.FL-R-SMT-1_Vertical
- J13: renamed from ?; value (none) -> JAE_SIM_Card_SF72S006; footprint (none) -> Connector_JAE:JAE_SIM_Card_SF72S006
- Q11, Q5, Q6, Q7, Q8, Q9: renamed from ?; value (none) -> NX3008NBKW; footprint (none) -> Package_TO_SOT_SMD:SOT-323_SC-70
- R18: renamed from ?; value (none) -> DNP; footprint (none) -> Resistor_SMD:R_0402_1005Metric
- R19, R20: renamed from ?; value (none) -> 0R; footprint (none) -> Resistor_SMD:R_0402_1005Metric
- R21, R33, R37, R38, R39, R40, R42, R43, R46: renamed from ?; value (none) -> 10k; footprint (none) -> Resistor_SMD:R_0603_1608Metric
- R22: renamed from ?; value (none) -> DNP 15k; footprint (none) -> Resistor_SMD:R_0603_1608Metric
- R23: renamed from ?; value (none) -> 0R; footprint (none) -> Resistor_SMD:R_0603_1608Metric
- R44: renamed from ?; value (none) -> 1k; footprint (none) -> Resistor_SMD:R_0603_1608Metric
- U7: renamed from ?; value (none) -> Sierra_Wireless_RC7620; footprint (none) -> jeffmakes-footprints:Cellular_Modem-Sierra-Wireless-module-CF3-ringCD
- U8: renamed from ?; value (none) -> ESD7004; footprint (none) -> Package_SON:USON-10_2.5x1.0mm_P0.5mm

Commit message: Set volage ratings on some caps, change some cap footprints to remove a couple of BOM lines
Parts:
- C22, C23: Voltage (none) -> 6.3V
- J1, J2, J3, J4, J5, J6, J7, J8, J9: now left out of the parts list
Changed lines of the file:
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@@
   )
   (symbol (lib_id "Connector:TestPoint") (at 170.18 161.29 270) (unit 1)
-    (in_bom yes) (on_board yes) (dnp no)
+    (in_bom no) (on_board yes) (dnp no)
     (property "Reference" "J2" (at 175.26 161.29 90)
       (effects (font (size 1.27 1.27)) (justify left))
@@
   )
   (symbol (lib_id "Connector:TestPoint") (at 170.18 171.45 270) (unit 1)
-    (in_bom yes) (on_board yes) (dnp no)
+    (in_bom no) (on_board yes) (dnp no)
     (property "Reference" "J6" (at 175.26 171.45 90)
       (effects (font (size 1.27 1.27)) (justify left))
@@
       (effects (font (size 1.27 1.27)) hide)
     )
+    (property "Voltage" "6.3V" (at 213.36 64.77 0)
+      (effects (font (size 1.27 1.27)) hide)
+    )
     (pin "1")
     (pin "2")
@@
   )
   (symbol (lib_id "Connector:TestPoint") (at 170.18 168.91 270) (unit 1)
-    (in_bom yes) (on_board yes) (dnp no)
+    (in_bom no) (on_board yes) (dnp no)
     (property "Reference" "J5" (at 175.26 168.91 90)
       (effects (font (size 1.27 1.27)) (justify left))
@@
   )
   (symbol (lib_id "Connector:TestPoint") (at 170.18 166.37 270) (unit 1)
-    (in_bom yes) (on_board yes) (dnp no)
+    (in_bom no) (on_board yes) (dnp no)
     (property "Reference" "J4" (at 175.26 166.37 90)
       (effects (font (size 1.27 1.27)) (justify left))
@@
   )
   (symbol (lib_id "Connector:TestPoint") (at 170.18 176.53 270) (unit 1)
-    (in_bom yes) (on_board yes) (dnp no)
+    (in_bom no) (on_board yes) (dnp no)
     (property "Reference" "J8" (at 175.26 176.53 90)
       (effects (font (size 1.27 1.27)) (justify left))
@@
   )
   (symbol (lib_id "Connector:TestPoint") (at 170.18 158.75 270) (unit 1)
-    (in_bom yes) (on_board yes) (dnp no)
+    (in_bom no) (on_board yes) (dnp no)
     (property "Reference" "J1" (at 175.26 158.75 90)
       (effects (font (size 1.27 1.27)) (justify left))
@@
   )
   (symbol (lib_id "Connector:TestPoint") (at 170.18 163.83 270) (unit 1)
-    (in_bom yes) (on_board yes) (dnp no)
+    (in_bom no) (on_board yes) (dnp no)
     (property "Reference" "J3" (at 175.26 163.83 90)
       (effects (font (size 1.27 1.27)) (justify left))
@@
     )
     (property "Datasheet" "~" (at 200.66 64.77 0)
+      (effects (font (size 1.27 1.27)) hide)
+    )
+    (property "Voltage" "6.3V" (at 200.66 64.77 0)
       (effects (font (size 1.27 1.27)) hide)
     )
@@
   )
   (symbol (lib_id "Connector:TestPoint") (at 170.18 173.99 270) (unit 1)
-    (in_bom yes) (on_board yes) (dnp no)
+    (in_bom no) (on_board yes) (dnp no)
     (property "Reference" "J7" (at 175.26 173.99 90)
       (effects (font (size 1.27 1.27)) (justify left))
@@
   )
   (symbol (lib_id "Connector:TestPoint") (at 170.18 179.07 270) (unit 1)
-    (in_bom yes) (on_board yes) (dnp no)
+    (in_bom no) (on_board yes) (dnp no)
     (property "Reference" "J9" (at 175.26 179.07 90)
       (effects (font (size 1.27 1.27)) (justify left))
