File: r4/src/_led_driver.kicad_sch (KiCad schematic)
At the start: 3 parts, among them J16 FH12A-20S-0.5SH, U9 PCF8574PW

Commit message: Update files to Kicad 6 format
Parts:
- ?: renamed from U9; value PCF8574PW -> (none); footprint Package_SO:SSOP-20_4.4x6.5mm_P0.65mm -> (none)
- ?: renamed from C38; value 100nF -> (none); footprint Capacitor_SMD:C_0603_1608Metric -> (none)
- ?: renamed from J16; value FH12A-20S-0.5SH -> (none); footprint Connector_FFC-FPC:Hirose_FH12-20S-0.5SH_1x20-1MP_P0.50mm_Horizontal -> (none)

Commit message: Add netclass definitions and assign nets. Define DRC rules to each class. Resize all vias and nets (with a few exceptions for very wide power tracks) to follow the netclass rules. Increase area for GNDA domain. Re-route SIM data bus around edge of GNDA domain
Parts:
- C38: renamed from ?; value (none) -> 100nF; footprint (none) -> Capacitor_SMD:C_0603_1608Metric
- J16: renamed from ?; value (none) -> FH12A-20S-0.5SH; footprint (none) -> Connector_FFC-FPC:Hirose_FH12-20S-0.5SH_1x20-1MP_P0.50mm_Horizontal
- U9: renamed from ?; value (none) -> PCF8574PW; footprint (none) -> Package_SO:SSOP-20_4.4x6.5mm_P0.65mm

Commit message: File noise due to Kicad version bump
Other:
- note added: "PCMD3180 Address 100 1100 (0x4C)"
Changed lines of the file:
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@@
-(kicad_sch (version 20221004) (generator eeschema)
+(kicad_sch (version 20230409) (generator eeschema)
   (paper "A4")
   (junction (at 127 67.31) (diameter 1.016) (color 0 0 0 0)
@@
     (stroke (width 0) (type solid))
   )
-  (text "Address 010 0011 (0x23)" (at 154.94 101.6 0)
+  (text "PCMD3180 Address 100 1100 (0x4C)" (exclude_from_sim no)
+ (at 229.87 91.44 0)
+    (effects (font (size 1.27 1.27)) (justify right bottom))
+  )
+  (text "Address 010 0011 (0x23)" (exclude_from_sim no)
+ (at 154.94 101.6 0)
     (effects (font (size 1.27 1.27)) (justify right bottom))
   )
@@
       (project "bugg-main-r4"
         (path "/e3eb514f-6ce4-4abe-ba20-f82f0015628f/676be2e4-179b-4538-a96d-4073cd6b4d31"
-          (reference "U9") (unit 1) (value "PCF8574PW") (footprint "Package_SO:SSOP-20_4.4x6.5mm_P0.65mm")
+          (reference "U9") (unit 1)
         )
       )
@@
       (project "bugg-main-r4"
         (path "/e3eb514f-6ce4-4abe-ba20-f82f0015628f/676be2e4-179b-4538-a96d-4073cd6b4d31"
-          (reference "#PWR0125") (unit 1) (value "GND") (footprint "")
+          (reference "#PWR0125") (unit 1)
         )
       )
@@
       (project "bugg-main-r4"
         (path "/e3eb514f-6ce4-4abe-ba20-f82f0015628f/676be2e4-179b-4538-a96d-4073cd6b4d31"
-          (reference "#PWR0127") (unit 1) (value "+3V3") (footprint "")
+          (reference "#PWR0127") (unit 1)
         )
       )
@@
       (project "bugg-main-r4"
         (path "/e3eb514f-6ce4-4abe-ba20-f82f0015628f/676be2e4-179b-4538-a96d-4073cd6b4d31"
-          (reference "#PWR0120") (unit 1) (value "GND") (footprint "")
+          (reference "#PWR0120") (unit 1)
         )
       )
@@
       (project "bugg-main-r4"
         (path "/e3eb514f-6ce4-4abe-ba20-f82f0015628f/676be2e4-179b-4538-a96d-4073cd6b4d31"
-          (reference "#PWR0114") (unit 1) (value "+3V3") (footprint "")
+          (reference "#PWR0114") (unit 1)
         )
       )
@@
       (project "bugg-main-r4"
         (path "/e3eb514f-6ce4-4abe-ba20-f82f0015628f/676be2e4-179b-4538-a96d-4073cd6b4d31"
-          (reference "#PWR0116") (unit 1) (value "+3V3") (footprint "")
+          (reference "#PWR0116") (unit 1)
         )
       )
@@
       (project "bugg-main-r4"
         (path "/e3eb514f-6ce4-4abe-ba20-f82f0015628f/676be2e4-179b-4538-a96d-4073cd6b4d31"
-          (reference "#PWR0124") (unit 1) (value "+5V") (footprint "")
+          (reference "#PWR0124") (unit 1)
         )
       )
@@
       (project "bugg-main-r4"
         (path "/e3eb514f-6ce4-4abe-ba20-f82f0015628f/676be2e4-179b-4538-a96d-4073cd6b4d31"
-          (reference "C38") (unit 1) (value "100nF") (footprint "Capacitor_SMD:C_0603_1608Metric")
+          (reference "C38") (unit 1)
         )
       )
@@
       (project "bugg-main-r4"
         (path "/e3eb514f-6ce4-4abe-ba20-f82f0015628f/676be2e4-179b-4538-a96d-4073cd6b4d31"
-          (reference "#PWR0117") (unit 1) (value "GND") (footprint "")
+          (reference "#PWR0117") (unit 1)
         )
       )
@@
       (project "bugg-main-r4"
         (path "/e3eb514f-6ce4-4abe-ba20-f82f0015628f/676be2e4-179b-4538-a96d-4073cd6b4d31"
-          (reference "#PWR0126") (unit 1) (value "+3V3") (footprint "")
+          (reference "#PWR0126") (unit 1)
         )
       )
@@
       (project "bugg-main-r4"
         (path "/e3eb514f-6ce4-4abe-ba20-f82f0015628f/676be2e4-179b-4538-a96d-4073cd6b4d31"
-          (reference "#PWR0112") (unit 1) (value "GND") (footprint "")
+          (reference "#PWR0112") (unit 1)
         )
       )
@@
       (project "bugg-main-r4"
         (path "/e3eb514f-6ce4-4abe-ba20-f82f0015628f/676be2e4-179b-4538-a96d-4073cd6b4d31"
-          (reference "#PWR0128") (unit 1) (value "GND") (footprint "")
+          (reference "#PWR0128") (unit 1)
         )
       )
@@
       (project "bugg-main-r4"
         (path "/e3eb514f-6ce4-4abe-ba20-f82f0015628f/676be2e4-179b-4538-a96d-4073cd6b4d31"
-          (reference "#PWR0122") (unit 1) (value "GND") (footprint "")
+          (reference "#PWR0122") (unit 1)
         )
       )
@@
       (project "bugg-main-r4"
         (path "/e3eb514f-6ce4-4abe-ba20-f82f0015628f/676be2e4-179b-4538-a96d-4073cd6b4d31"
-          (reference "J16") (unit 1) (value "FH12A-20S-0.5SH") (footprint "Connector_FFC-FPC:Hirose_FH12-20S-0.5SH_1x20-1MP_P0.50mm_Horizontal")
-        )
-      )
+          (reference "J16") (unit 1)
+        )
+      )

Commit message: Create new branch for next schematic revision. Move PCF8574 to 5.4V rail and add level translator circuit to convert the 3.3V I2C bus up to 5V. This fixes the problem of the red LED's being impossible to fully turn off because their cathodes can only get up to 3.3V and so they have 5.4-3.3=2.1V across them permanently in the current design
Parts:
- added Q22 (x2): NX3008NBKW, Package_TO_SOT_SMD:SOT-323_SC-70, symbol Device:Q_NMOS_GSD
- added R33 (x2): 10k, Resistor_SMD:R_0402_1005Metric, symbol Device:R_Small
Connections:
- net +3V3: now also Q22.1 (G), Q22.1 (G); no longer C38.2, U9.5 (VDD), U9.6 (A0), U9.7 (A1)
- net +5V: now also C38.2, U9.5 (VDD), U9.6 (A0), U9.7 (A1), R33.1, R33.1
- net SCL: now also Q22.2 (S); no longer U9.2 (SCL)
- net SDA: now also Q22.2 (S); no longer U9.4 (SDA)
- new net SCL_5V: Q22.3 (D), R33.2, U9.2 (SCL)
- new net SDA_5V: Q22.3 (D), R33.2, U9.4 (SDA)
Other:
- note added: "Level translator per NXP AN10441"
