File: r5/src/_led_driver.kicad_sch (KiCad schematic)
At the start: 7 parts, among them J16 FH12A-20S-0.5SH, Q22 NX3008NBKW, U9 PCF8574PW

Commit message: Oops, hadn't run the ERC for ages. Ran, passed. Add ERC and DRC exclusions where unavoidable
Parts:
- J16: Digikey (none) -> HFK120CT-ND; MPN (none) -> FH12A-20S-0.5SH(55); Manufacturer (none) -> Hirose; Mouser (none) -> 798-FH12A-20S0.5SH55
- Q22: Digikey (none) -> 1727-1280-6-ND; MPN (none) -> NX3008NBKW; Manufacturer (none) -> Nexperia; Mouser (none) -> 771-NX3008NBKW,115
- U9: Digikey (none) -> TI; MPN (none) -> PCF8574PW; Manufacturer (none) -> TI; Mouser (none) -> 595-PCF8574PWG4
Changed lines of the file:
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@@
-      (effects (font (size 1.27 1.27)) hide)
-    )
-    (property "MANUFACTURER" "" (at 142.24 69.85 0)
       (effects (font (size 1.27 1.27)) hide)
     )
@@
       (effects (font (size 1.27 1.27)) hide)
     )
-    (property "Digikey" "" (at 142.24 69.85 0)
-      (effects (font (size 1.27 1.27)) hide)
-    )
-    (property "MPN" "" (at 142.24 69.85 0)
-      (effects (font (size 1.27 1.27)) hide)
-    )
-    (property "Mouser" "" (at 142.24 69.85 0)
+    (property "Digikey" "TI" (at 142.24 69.85 0)
+      (effects (font (size 1.27 1.27)) hide)
+    )
+    (property "MPN" "PCF8574PW " (at 142.24 69.85 0)
+      (effects (font (size 1.27 1.27)) hide)
+    )
+    (property "Mouser" "595-PCF8574PWG4" (at 142.24 69.85 0)
+      (effects (font (size 1.27 1.27)) hide)
+    )
+    (property "Farnell" "" (at 142.24 69.85 0)
       (effects (font (size 1.27 1.27)) hide)
     )
     (property "Field-1" "" (at 142.24 69.85 0)
+      (effects (font (size 1.27 1.27)) hide)
+    )
+    (property "Manufacturer" "TI" (at 142.24 69.85 0)
       (effects (font (size 1.27 1.27)) hide)
     )
@@
       (effects (font (size 1.27 1.27)) hide)
     )
-    (property "MANUFACTURER" "" (at 97.79 57.15 0)
-      (effects (font (size 1.27 1.27)) hide)
-    )
     (property "Quantity" "" (at 97.79 57.15 0)
       (effects (font (size 1.27 1.27)) hide)
@@
     )
     (property "Mouser" "" (at 97.79 57.15 0)
+      (effects (font (size 1.27 1.27)) hide)
+    )
+    (property "Farnell" "" (at 97.79 57.15 0)
       (effects (font (size 1.27 1.27)) hide)
     )
@@
       (effects (font (size 1.27 1.27)) hide)
     )
-    (property "MANUFACTURER" "" (at 76.2 59.69 0)
-      (effects (font (size 1.27 1.27)) hide)
-    )
     (property "Quantity" "" (at 76.2 59.69 0)
       (effects (font (size 1.27 1.27)) hide)
     )
-    (property "Digikey" "" (at 76.2 59.69 0)
-      (effects (font (size 1.27 1.27)) hide)
-    )
-    (property "MPN" "" (at 76.2 59.69 0)
-      (effects (font (size 1.27 1.27)) hide)
-    )
-    (property "Mouser" "" (at 76.2 59.69 0)
+    (property "Digikey" "1727-1280-6-ND" (at 76.2 59.69 0)
+      (effects (font (size 1.27 1.27)) hide)
+    )
+    (property "MPN" "NX3008NBKW" (at 76.2 59.69 0)
+      (effects (font (size 1.27 1.27)) hide)
+    )
+    (property "Mouser" "771-NX3008NBKW,115" (at 76.2 59.69 0)
+      (effects (font (size 1.27 1.27)) hide)
+    )
+    (property "Farnell" "" (at 76.2 59.69 0)
       (effects (font (size 1.27 1.27)) hide)
     )
     (property "Field-1" "" (at 76.2 59.69 0)
+      (effects (font (size 1.27 1.27)) hide)
+    )
+    (property "Manufacturer" "Nexperia" (at 76.2 59.69 0)
       (effects (font (size 1.27 1.27)) hide)
     )
@@
       (effects (font (size 1.27 1.27)) hide)
     )
-    (property "MANUFACTURER" "" (at 97.79 43.18 0)
-      (effects (font (size 1.27 1.27)) hide)
-    )
     (property "Quantity" "" (at 97.79 43.18 0)
       (effects (font (size 1.27 1.27)) hide)
@@
     )
     (property "Mouser" "" (at 97.79 43.18 0)
+      (effects (font (size 1.27 1.27)) hide)
+    )
+    (property "Farnell" "" (at 97.79 43.18 0)
       (effects (font (size 1.27 1.27)) hide)
     )
@@
       (effects (font (size 1.27 1.27)) hide)
     )
-    (property "MANUFACTURER" "" (at 134.62 43.18 0)
-      (effects (font (size 1.27 1.27)) hide)
-    )
     (property "Quantity" "" (at 134.62 43.18 0)
       (effects (font (size 1.27 1.27)) hide)
@@
       (effects (font (size 1.27 1.27)) hide)
     )
+    (property "Manufacturer" "Murata" (at 134.62 43.18 0)
+      (effects (font (size 1.27 1.27)) hide)
+    )
+    (property "Voltage" "50V" (at 134.62 43.18 0)
+      (effects (font (size 1.27 1.27)) hide)
+    )
+    (property "Farnell" "" (at 134.62 43.18 0)
+      (effects (font (size 1.27 1.27)) hide)
+    )
     (property "Field-1" "" (at 134.62 43.18 0)
-      (effects (font (size 1.27 1.27)) hide)
-    )
-    (property "Manufacturer" "Murata" (at 134.62 43.18 0)
-      (effects (font (size 1.27 1.27)) hide)
-    )
-    (property "Voltage" "50V" (at 134.62 43.18 0)
       (effects (font (size 1.27 1.27)) hide)
     )
@@
       (effects (font (size 1.27 1.27)) hide)
     )
-    (property "MANUFACTURER" "" (at 76.2 45.72 0)
-      (effects (font (size 1.27 1.27)) hide)
-    )
     (property "Quantity" "" (at 76.2 45.72 0)
       (effects (font (size 1.27 1.27)) hide)
     )
-    (property "Digikey" "" (at 76.2 45.72 0)
-      (effects (font (size 1.27 1.27)) hide)
-    )
-    (property "MPN" "" (at 76.2 45.72 0)
-      (effects (font (size 1.27 1.27)) hide)
-    )
-    (property "Mouser" "" (at 76.2 45.72 0)
+    (property "Digikey" "1727-1280-6-ND" (at 76.2 45.72 0)
+      (effects (font (size 1.27 1.27)) hide)
+    )
+    (property "MPN" "NX3008NBKW" (at 76.2 45.72 0)
+      (effects (font (size 1.27 1.27)) hide)
+    )
+    (property "Mouser" "771-NX3008NBKW,115" (at 76.2 45.72 0)
+      (effects (font (size 1.27 1.27)) hide)
+    )
+    (property "Farnell" "" (at 76.2 45.72 0)
       (effects (font (size 1.27 1.27)) hide)
     )
     (property "Field-1" "" (at 76.2 45.72 0)
+      (effects (font (size 1.27 1.27)) hide)
+    )
+    (property "Manufacturer" "Nexperia" (at 76.2 45.72 0)
       (effects (font (size 1.27 1.27)) hide)
     )
@@
       (effects (font (size 1.27 1.27)) hide)
     )
-    (property "MANUFACTURER" "" (at 189.23 72.39 0)
-      (effects (font (size 1.27 1.27)) hide)
-    )
     (property "Quantity" "" (at 189.23 72.39 0)
       (effects (font (size 1.27 1.27)) hide)
     )
-    (property "Digikey" "" (at 189.23 72.39 0)
-      (effects (font (size 1.27 1.27)) hide)
-    )
-    (property "MPN" "" (at 189.23 72.39 0)
-      (effects (font (size 1.27 1.27)) hide)
-    )
-    (property "Mouser" "" (at 189.23 72.39 0)
-      (effects (font (size 1.27 1.27)) hide)
-    )
+    (property "Digikey" "HFK120CT-ND" (at 189.23 72.39 0)
+      (effects (font (size 1.27 1.27)) hide)
+    )
+    (property "MPN" "FH12A-20S-0.5SH(55)" (at 189.23 72.39 0)
+      (effects (font (size 1.27 1.27)) hide)
+    )
+    (property "Mouser" "798-FH12A-20S0.5SH55" (at 189.23 72.39 0)
+      (effects (font (size 1.27 1.27)) hide)
+    )
+    (property "Manufacturer" "Hirose" (at 189.23 72.39 0)
+      (effects (font (size 1.27 1.27)) hide)
+    )
+    (property "Farnell" "" (at 189.23 72.39 0)
+      (effects (font (size 1.27 1.27)) hide)
+    )
