File: r5/src/_usb-serial.kicad_sch (KiCad schematic)
At the start: 13 parts, among them T41 , U12 CP2102N-Axx-xQFN24

Commit message: Oops, hadn't run the ERC for ages. Ran, passed. Add ERC and DRC exclusions where unavoidable
Parts:
- U12: Digikey (none) -> 336-5888-6-ND; MPN (none) -> CP2102N-A02-GQFN24R; Manufacturer (none) -> Si Labs; Mouser (none) -> 634-CP2102NA02QFN24R
Changed lines of the file:
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@@
-      (effects (font (size 1.27 1.27)) hide)
-    )
-    (property "MANUFACTURER" "" (at 127 74.93 0)
       (effects (font (size 1.27 1.27)) hide)
     )
@@
       (effects (font (size 1.27 1.27)) hide)
     )
+    (property "Farnell" "" (at 127 74.93 0)
+      (effects (font (size 1.27 1.27)) hide)
+    )
     (property "Field-1" "" (at 127 74.93 0)
       (effects (font (size 1.27 1.27)) hide)
@@
       (effects (font (size 1.27 1.27)) hide)
     )
-    (property "MANUFACTURER" "" (at 154.94 62.23 0)
-      (effects (font (size 1.27 1.27)) hide)
-    )
     (property "Quantity" "" (at 154.94 62.23 0)
       (effects (font (size 1.27 1.27)) hide)
@@
       (effects (font (size 1.27 1.27)) hide)
     )
+    (property "Manufacturer" "Murata" (at 154.94 62.23 0)
+      (effects (font (size 1.27 1.27)) hide)
+    )
+    (property "Voltage" "50V" (at 154.94 62.23 0)
+      (effects (font (size 1.27 1.27)) hide)
+    )
+    (property "Farnell" "" (at 154.94 62.23 0)
+      (effects (font (size 1.27 1.27)) hide)
+    )
     (property "Field-1" "" (at 154.94 62.23 0)
       (effects (font (size 1.27 1.27)) hide)
     )
-    (property "Manufacturer" "Murata" (at 154.94 62.23 0)
-      (effects (font (size 1.27 1.27)) hide)
-    )
-    (property "Voltage" "50V" (at 154.94 62.23 0)
-      (effects (font (size 1.27 1.27)) hide)
-    )
     (pin "1")
     (pin "2")
@@
       (effects (font (size 1.27 1.27)) hide)
     )
-    (property "MANUFACTURER" "" (at 168.91 62.23 0)
-      (effects (font (size 1.27 1.27)) hide)
-    )
     (property "Quantity" "" (at 168.91 62.23 0)
       (effects (font (size 1.27 1.27)) hide)
@@
       (effects (font (size 1.27 1.27)) hide)
     )
+    (property "Farnell" "" (at 168.91 62.23 0)
+      (effects (font (size 1.27 1.27)) hide)
+    )
     (property "Field-1" "" (at 168.91 62.23 0)
       (effects (font (size 1.27 1.27)) hide)
@@
       (effects (font (size 1.27 1.27)) hide)
     )
-    (property "MANUFACTURER" "" (at 205.74 80.01 0)
-      (effects (font (size 1.27 1.27)) hide)
-    )
     (property "Quantity" "" (at 205.74 80.01 0)
       (effects (font (size 1.27 1.27)) hide)
@@
       (effects (font (size 1.27 1.27)) hide)
     )
+    (property "Manufacturer" "Murata" (at 205.74 80.01 0)
+      (effects (font (size 1.27 1.27)) hide)
+    )
+    (property "Voltage" "50V" (at 205.74 80.01 0)
+      (effects (font (size 1.27 1.27)) hide)
+    )
+    (property "Farnell" "" (at 205.74 80.01 0)
+      (effects (font (size 1.27 1.27)) hide)
+    )
     (property "Field-1" "" (at 205.74 80.01 0)
       (effects (font (size 1.27 1.27)) hide)
     )
-    (property "Manufacturer" "Murata" (at 205.74 80.01 0)
-      (effects (font (size 1.27 1.27)) hide)
-    )
-    (property "Voltage" "50V" (at 205.74 80.01 0)
-      (effects (font (size 1.27 1.27)) hide)
-    )
     (pin "1")
     (pin "2")
@@
       (effects (font (size 1.27 1.27)) hide)
     )
-    (property "MANUFACTURER" "" (at 179.07 80.01 0)
-      (effects (font (size 1.27 1.27)) hide)
-    )
     (property "Quantity" "" (at 179.07 80.01 0)
       (effects (font (size 1.27 1.27)) hide)
@@
       (effects (font (size 1.27 1.27)) hide)
     )
+    (property "Manufacturer" "Murata" (at 179.07 80.01 0)
+      (effects (font (size 1.27 1.27)) hide)
+    )
+    (property "Voltage" "50V" (at 179.07 80.01 0)
+      (effects (font (size 1.27 1.27)) hide)
+    )
+    (property "Farnell" "" (at 179.07 80.01 0)
+      (effects (font (size 1.27 1.27)) hide)
+    )
     (property "Field-1" "" (at 179.07 80.01 0)
       (effects (font (size 1.27 1.27)) hide)
     )
-    (property "Manufacturer" "Murata" (at 179.07 80.01 0)
-      (effects (font (size 1.27 1.27)) hide)
-    )
-    (property "Voltage" "50V" (at 179.07 80.01 0)
-      (effects (font (size 1.27 1.27)) hide)
-    )
     (pin "1")
     (pin "2")
@@
       (effects (font (size 1.27 1.27)) hide)
     )
-    (property "MANUFACTURER" "" (at 120.65 110.49 0)
-      (effects (font (size 1.27 1.27)) hide)
-    )
     (property "Quantity" "" (at 120.65 110.49 0)
       (effects (font (size 1.27 1.27)) hide)
@@
       (effects (font (size 1.27 1.27)) hide)
     )
+    (property "Farnell" "" (at 120.65 110.49 0)
+      (effects (font (size 1.27 1.27)) hide)
+    )
     (property "Field-1" "" (at 120.65 110.49 0)
       (effects (font (size 1.27 1.27)) hide)
@@
       (effects (font (size 1.27 1.27)) hide)
     )
-    (property "MANUFACTURER" "" (at 120.65 93.98 0)
-      (effects (font (size 1.27 1.27)) hide)
-    )
     (property "Quantity" "" (at 120.65 93.98 0)
       (effects (font (size 1.27 1.27)) hide)
@@
       (effects (font (size 1.27 1.27)) hide)
     )
+    (property "Farnell" "" (at 120.65 93.98 0)
+      (effects (font (size 1.27 1.27)) hide)
+    )
     (property "Field-1" "" (at 120.65 93.98 0)
       (effects (font (size 1.27 1.27)) hide)
@@
       (effects (font (size 1.27 1.27)) hide)
     )
-    (property "MANUFACTURER" "" (at 214.63 80.01 0)
-      (effects (font (size 1.27 1.27)) hide)
-    )
     (property "Quantity" "" (at 214.63 80.01 0)
       (effects (font (size 1.27 1.27)) hide)
@@
       (effects (font (size 1.27 1.27)) hide)
     )
+    (property "Manufacturer" "Murata" (at 214.63 80.01 0)
+      (effects (font (size 1.27 1.27)) hide)
+    )
+    (property "Farnell" "" (at 214.63 80.01 0)
+      (effects (font (size 1.27 1.27)) hide)
+    )
     (property "Field-1" "" (at 214.63 80.01 0)
       (effects (font (size 1.27 1.27)) hide)
     )
-    (property "Manufacturer" "Murata" (at 214.63 80.01 0)
-      (effects (font (size 1.27 1.27)) hide)
-    )
     (pin "1")
     (pin "2")
@@
       (effects (font (size 1.27 1.27)) hide)
     )
-    (property "MANUFACTURER" "" (at 160.02 85.09 0)
-      (effects (font (size 1.27 1.27)) hide)
-    )
     (property "Quantity" "" (at 160.02 85.09 0)
       (effects (font (size 1.27 1.27)) hide)
@@
     )
     (property "Mouser" "" (at 160.02 85.09 0)
+      (effects (font (size 1.27 1.27)) hide)
+    )
+    (property "Farnell" "" (at 160.02 85.09 0)
       (effects (font (size 1.27 1.27)) hide)
     )
@@
       (effects (font (size 1.27 1.27)) hide)
     )
-    (property "MANUFACTURER" "" (at 120.65 116.84 0)
-      (effects (font (size 1.27 1.27)) hide)
-    )
     (property "Quantity" "" (at 120.65 116.84 0)
       (effects (font (size 1.27 1.27)) hide)
@@
       (effects (font (size 1.27 1.27)) hide)
     )
+    (property "Farnell" "" (at 120.65 116.84 0)
+      (effects (font (size 1.27 1.27)) hide)
+    )
     (property "Field-1" "" (at 120.65 116.84 0)
       (effects (font (size 1.27 1.27)) hide)
@@
       (effects (font (size 1.27 1.27)) hide)
     )
-    (property "MANUFACTURER" "" (at 143.51 110.49 0)
-      (effects (font (size 1.27 1.27)) hide)
-    )
     (property "Quantity" "" (at 143.51 110.49 0)
       (effects (font (size 1.27 1.27)) hide)
     )
-    (property "Digikey" "" (at 143.51 110.49 0)
-      (effects (font (size 1.27 1.27)) hide)
-    )
-    (property "MPN" "" (at 143.51 110.49 0)
-      (effects (font (size 1.27 1.27)) hide)
-    )
-    (property "Mouser" "" (at 143.51 110.49 0)
+    (property "Digikey" "336-5888-6-ND" (at 143.51 110.49 0)
+      (effects (font (size 1.27 1.27)) hide)
+    )
+    (property "MPN" "CP2102N-A02-GQFN24R" (at 143.51 110.49 0)
+      (effects (font (size 1.27 1.27)) hide)
+    )
+    (property "Mouser" "634-CP2102NA02QFN24R" (at 143.51 110.49 0)
+      (effects (font (size 1.27 1.27)) hide)
+    )
+    (property "Farnell" "" (at 143.51 110.49 0)
       (effects (font (size 1.27 1.27)) hide)
     )
     (property "Field-1" "" (at 143.51 110.49 0)
+      (effects (font (size 1.27 1.27)) hide)
+    )
+    (property "Manufacturer" "Si Labs" (at 143.51 110.49 0)
       (effects (font (size 1.27 1.27)) hide)
     )
@@
       (effects (font (size 1.27 1.27)) hide)
     )
-    (property "MANUFACTURER" "" (at 187.96 80.01 0)
-      (effects (font (size 1.27 1.27)) hide)
-    )
     (property "Quantity" "" (at 187.96 80.01 0)
       (effects (font (size 1.27 1.27)) hide)
@@
       (effects (font (size 1.27 1.27)) hide)
     )
+    (property "Manufacturer" "Murata" (at 187.96 80.01 0)
+      (effects (font (size 1.27 1.27)) hide)
+    )
+    (property "Farnell" "" (at 187.96 80.01 0)
+      (effects (font (size 1.27 1.27)) hide)
+    )
     (property "Field-1" "" (at 187.96 80.01 0)
       (effects (font (size 1.27 1.27)) hide)
     )
-    (property "Manufacturer" "Murata" (at 187.96 80.01 0)
-      (effects (font (size 1.27 1.27)) hide)
-    )
     (pin "1")
     (pin "2")
@@
       (effects (font (size 1.27 1.27)) hide)
     )
-    (property "MANUFACTURER" "" (at 162.56 85.09 0)
-      (effects (font (size 1.27 1.27)) hide)
-    )
     (property "Quantity" "" (at 162.56 85.09 0)
       (effects (font (size 1.27 1.27)) hide)
@@
       (effects (font (size 1.27 1.27)) hide)
     )
+    (property "Farnell" "" (at 162.56 85.09 0)
+      (effects (font (size 1.27 1.27)) hide)
+    )
