File: r5/src/_usb_otg.kicad_sch (KiCad schematic)
At the start: 7 parts, among them J15 10118194, Q4 NX3008NBKW, U15 FSUSB42MX, U16 ESD7004

Commit message: Updates to +/-15V supply. Additional output capacitance. Change to smaller inductor packages. Add 0R links to permit isolation of output. Mods to compensation network. Set feedback resistors to datasheet values.
Parts:
- renumbered C37 to C93, Q4 to Q11, R31 to R63, R32 to R64, U15 to U22, U16 to U23
Changed lines of the file:
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@@
   (symbol (lib_id "j_Power_Protection:ESD7004") (at 172.72 120.65 0) (unit 1)
     (in_bom yes) (on_board yes) (dnp no)
-    (property "Reference" "U16" (at 180.34 118.11 0)
+    (property "Reference" "U23" (at 180.34 118.11 0)
       (effects (font (size 1.27 1.27)) (justify left))
     )
@@
       (project "bugg-main-r5"
         (path "/e3eb514f-6ce4-4abe-ba20-f82f0015628f/7086fb34-03e0-4978-93d2-ceae572d34d4"
-          (reference "U16") (unit 1)
+          (reference "U23") (unit 1)
         )
       )
@@
   (symbol (lib_id "power:GND") (at 172.72 125.73 0) (unit 1)
     (in_bom yes) (on_board yes) (dnp no)
-    (property "Reference" "#PWR0110" (at 172.72 132.08 0)
+    (property "Reference" "#PWR0184" (at 172.72 132.08 0)
       (effects (font (size 1.27 1.27)) hide)
     )
@@
       (project "bugg-main-r5"
         (path "/e3eb514f-6ce4-4abe-ba20-f82f0015628f/7086fb34-03e0-4978-93d2-ceae572d34d4"
-          (reference "#PWR0110") (unit 1)
+          (reference "#PWR0184") (unit 1)
         )
       )
@@
   (symbol (lib_id "power:GND") (at 118.11 90.17 0) (unit 1)
     (in_bom yes) (on_board yes) (dnp no)
-    (property "Reference" "#PWR0107" (at 118.11 96.52 0)
+    (property "Reference" "#PWR0181" (at 118.11 96.52 0)
       (effects (font (size 1.27 1.27)) hide)
     )
@@
       (project "bugg-main-r5"
         (path "/e3eb514f-6ce4-4abe-ba20-f82f0015628f/7086fb34-03e0-4978-93d2-ceae572d34d4"
-          (reference "#PWR0107") (unit 1)
+          (reference "#PWR0181") (unit 1)
         )
       )
@@
   (symbol (lib_id "CM4IO:FSUSB42MX") (at 132.08 110.49 0) (mirror y) (unit 1)
     (in_bom yes) (on_board yes) (dnp no)
-    (property "Reference" "U15" (at 133.35 86.995 0)
+    (property "Reference" "U22" (at 133.35 86.995 0)
       (effects (font (size 1.27 1.27)))
     )
@@
       (project "bugg-main-r5"
         (path "/e3eb514f-6ce4-4abe-ba20-f82f0015628f/7086fb34-03e0-4978-93d2-ceae572d34d4"
-          (reference "U15") (unit 1)
+          (reference "U22") (unit 1)
         )
       )
@@
   (symbol (lib_id "Device:C_Small") (at 118.11 87.63 180) (unit 1)
     (in_bom yes) (on_board yes) (dnp no)
-    (property "Reference" "C37" (at 110.49 86.36 0)
+    (property "Reference" "C93" (at 110.49 86.36 0)
       (effects (font (size 1.27 1.27)) (justify right))
     )
@@
       (project "bugg-main-r5"
         (path "/e3eb514f-6ce4-4abe-ba20-f82f0015628f/7086fb34-03e0-4978-93d2-ceae572d34d4"
-          (reference "C37") (unit 1)
+          (reference "C93") (unit 1)
         )
       )
@@
   (symbol (lib_id "power:GND") (at 161.29 83.82 0) (unit 1)
     (in_bom yes) (on_board yes) (dnp no)
-    (property "Reference" "#PWR0109" (at 161.29 90.17 0)
+    (property "Reference" "#PWR0183" (at 161.29 90.17 0)
       (effects (font (size 1.27 1.27)) hide)
     )
@@
       (project "bugg-main-r5"
         (path "/e3eb514f-6ce4-4abe-ba20-f82f0015628f/7086fb34-03e0-4978-93d2-ceae572d34d4"
-          (reference "#PWR0109") (unit 1)
+          (reference "#PWR0183") (unit 1)
         )
       )
@@
   (symbol (lib_id "power:+3V3") (at 118.11 82.55 0) (unit 1)
     (in_bom yes) (on_board yes) (dnp no)
-    (property "Reference" "#PWR0106" (at 118.11 86.36 0)
+    (property "Reference" "#PWR0180" (at 118.11 86.36 0)
       (effects (font (size 1.27 1.27)) hide)
     )
@@
       (project "bugg-main-r5"
         (path "/e3eb514f-6ce4-4abe-ba20-f82f0015628f/7086fb34-03e0-4978-93d2-ceae572d34d4"
-          (reference "#PWR0106") (unit 1)
+          (reference "#PWR0180") (unit 1)
         )
       )
@@
   (symbol (lib_id "power:GND") (at 109.22 113.03 0) (unit 1)
     (in_bom yes) (on_board yes) (dnp no)
-    (property "Reference" "#PWR0105" (at 109.22 119.38 0)
+    (property "Reference" "#PWR0179" (at 109.22 119.38 0)
       (effects (font (size 1.27 1.27)) hide)
     )
@@
       (project "bugg-main-r5"
         (path "/e3eb514f-6ce4-4abe-ba20-f82f0015628f/7086fb34-03e0-4978-93d2-ceae572d34d4"
-          (reference "#PWR0105") (unit 1)
+          (reference "#PWR0179") (unit 1)
         )
       )
@@
   (symbol (lib_id "power:GND") (at 207.01 120.65 0) (unit 1)
     (in_bom yes) (on_board yes) (dnp no)
-    (property "Reference" "#PWR0111" (at 207.01 127 0)
+    (property "Reference" "#PWR0185" (at 207.01 127 0)
       (effects (font (size 1.27 1.27)) hide)
     )
@@
       (project "bugg-main-r5"
         (path "/e3eb514f-6ce4-4abe-ba20-f82f0015628f/7086fb34-03e0-4978-93d2-ceae572d34d4"
-          (reference "#PWR0111") (unit 1)
+          (reference "#PWR0185") (unit 1)
         )
       )
@@
   (symbol (lib_id "power:GND") (at 120.65 113.03 0) (unit 1)
     (in_bom yes) (on_board yes) (dnp no)
-    (property "Reference" "#PWR0108" (at 120.65 119.38 0)
+    (property "Reference" "#PWR0182" (at 120.65 119.38 0)
       (effects (font (size 1.27 1.27)) hide)
     )
@@
       (project "bugg-main-r5"
         (path "/e3eb514f-6ce4-4abe-ba20-f82f0015628f/7086fb34-03e0-4978-93d2-ceae572d34d4"
-          (reference "#PWR0108") (unit 1)
+          (reference "#PWR0182") (unit 1)
         )
       )
@@
   (symbol (lib_id "Device:R_Small") (at 109.22 109.22 0) (unit 1)
     (in_bom yes) (on_board yes) (dnp no)
-    (property "Reference" "R32" (at 111.125 108.585 0)
+    (property "Reference" "R64" (at 111.125 108.585 0)
       (effects (font (size 1.27 1.27)) (justify left))
     )
@@
       (project "bugg-main-r5"
         (path "/e3eb514f-6ce4-4abe-ba20-f82f0015628f/7086fb34-03e0-4978-93d2-ceae572d34d4"
-          (reference "R32") (unit 1)
+          (reference "R64") (unit 1)
         )
       )
@@
   (symbol (lib_id "Device:R_Small") (at 106.68 85.09 0) (mirror x) (unit 1)
     (in_bom yes) (on_board yes) (dnp no)
-    (property "Reference" "R31" (at 104.14 83.82 0)
+    (property "Reference" "R63" (at 104.14 83.82 0)
       (effects (font (size 1.27 1.27)) (justify right))
     )
@@
       (project "bugg-main-r5"
         (path "/e3eb514f-6ce4-4abe-ba20-f82f0015628f/7086fb34-03e0-4978-93d2-ceae572d34d4"
-          (reference "R31") (unit 1)
+          (reference "R63") (unit 1)
         )
       )
@@
   (symbol (lib_id "Device:Q_NMOS_GSD") (at 158.75 78.74 0) (unit 1)
     (in_bom yes) (on_board yes) (dnp no)
-    (property "Reference" "Q4" (at 165.1 77.47 0)
+    (property "Reference" "Q11" (at 165.1 77.47 0)
       (effects (font (size 1.27 1.27)) (justify left))
     )
@@
       (project "bugg-main-r5"
         (path "/e3eb514f-6ce4-4abe-ba20-f82f0015628f/7086fb34-03e0-4978-93d2-ceae572d34d4"
-          (reference "Q4") (unit 1)
-        )
-      )
+          (reference "Q11") (unit 1)
+        )
+      )

Commit message: Fix broken component annotation by importing back from PCB and fixing duplicates.
Parts:
- renumbered C93 to C37, Q11 to Q4, R63 to R31, R64 to R32, U22 to U15, U23 to U16
Changed lines of the file:
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@@
   (symbol (lib_id "j_Power_Protection:ESD7004") (at 172.72 120.65 0) (unit 1)
     (in_bom yes) (on_board yes) (dnp no)
-    (property "Reference" "U23" (at 180.34 118.11 0)
+    (property "Reference" "U16" (at 180.34 118.11 0)
       (effects (font (size 1.27 1.27)) (justify left))
     )
@@
       (project "bugg-main-r5"
         (path "/e3eb514f-6ce4-4abe-ba20-f82f0015628f/7086fb34-03e0-4978-93d2-ceae572d34d4"
-          (reference "U23") (unit 1)
+          (reference "U16") (unit 1)
         )
       )
@@
   (symbol (lib_id "CM4IO:FSUSB42MX") (at 132.08 110.49 0) (mirror y) (unit 1)
     (in_bom yes) (on_board yes) (dnp no)
-    (property "Reference" "U22" (at 133.35 86.995 0)
+    (property "Reference" "U15" (at 133.35 86.995 0)
       (effects (font (size 1.27 1.27)))
     )
@@
       (project "bugg-main-r5"
         (path "/e3eb514f-6ce4-4abe-ba20-f82f0015628f/7086fb34-03e0-4978-93d2-ceae572d34d4"
-          (reference "U22") (unit 1)
+          (reference "U15") (unit 1)
         )
       )
@@
   (symbol (lib_id "Device:C_Small") (at 118.11 87.63 180) (unit 1)
     (in_bom yes) (on_board yes) (dnp no)
-    (property "Reference" "C93" (at 110.49 86.36 0)
+    (property "Reference" "C37" (at 110.49 86.36 0)
       (effects (font (size 1.27 1.27)) (justify right))
     )
@@
       (project "bugg-main-r5"
         (path "/e3eb514f-6ce4-4abe-ba20-f82f0015628f/7086fb34-03e0-4978-93d2-ceae572d34d4"
-          (reference "C93") (unit 1)
+          (reference "C37") (unit 1)
         )
       )
@@
   (symbol (lib_id "Device:R_Small") (at 109.22 109.22 0) (unit 1)
     (in_bom yes) (on_board yes) (dnp no)
-    (property "Reference" "R64" (at 111.125 108.585 0)
+    (property "Reference" "R32" (at 111.125 108.585 0)
       (effects (font (size 1.27 1.27)) (justify left))
     )
@@
       (project "bugg-main-r5"
         (path "/e3eb514f-6ce4-4abe-ba20-f82f0015628f/7086fb34-03e0-4978-93d2-ceae572d34d4"
-          (reference "R64") (unit 1)
+          (reference "R32") (unit 1)
         )
       )
@@
   (symbol (lib_id "Device:R_Small") (at 106.68 85.09 0) (mirror x) (unit 1)
     (in_bom yes) (on_board yes) (dnp no)
-    (property "Reference" "R63" (at 104.14 83.82 0)
+    (property "Reference" "R31" (at 104.14 83.82 0)
       (effects (font (size 1.27 1.27)) (justify right))
     )
@@
       (project "bugg-main-r5"
         (path "/e3eb514f-6ce4-4abe-ba20-f82f0015628f/7086fb34-03e0-4978-93d2-ceae572d34d4"
-          (reference "R63") (unit 1)
+          (reference "R31") (unit 1)
         )
       )
@@
   (symbol (lib_id "Device:Q_NMOS_GSD") (at 158.75 78.74 0) (unit 1)
     (in_bom yes) (on_board yes) (dnp no)
-    (property "Reference" "Q11" (at 165.1 77.47 0)
+    (property "Reference" "Q4" (at 165.1 77.47 0)
       (effects (font (size 1.27 1.27)) (justify left))
     )
@@
       (project "bugg-main-r5"
         (path "/e3eb514f-6ce4-4abe-ba20-f82f0015628f/7086fb34-03e0-4978-93d2-ceae572d34d4"
-          (reference "Q11") (unit 1)
-        )
-      )
+          (reference "Q4") (unit 1)
+        )
+      )

Commit message: Update layout to standardise on 0402 passives everywhere possible. This reduces the number of BoM lines. DRC passed. Add DRC exclusions for unavoidable violations
Parts:
- C37: footprint Capacitor_SMD:C_0603_1608Metric -> Capacitor_SMD:C_0402_1005Metric
Changed lines of the file:
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@@
       (effects (font (size 1.27 1.27)) (justify right))
     )
-    (property "Footprint" "Capacitor_SMD:C_0603_1608Metric" (at 118.11 87.63 0)
+    (property "Footprint" "Capacitor_SMD:C_0402_1005Metric" (at 118.11 87.63 0)
       (effects (font (size 1.27 1.27)) hide)
     )

Commit message: Change 0805 47uF to 1206 to save a BOM line. Update layout, DRC pass.
Parts:
- C37: MPN (none) -> GRM155R71H104KE14D; Manufacturer (none) -> Murata; Mouser (none) -> 81-GRM155R71H104KE4D; Voltage (none) -> 50V
Changed lines of the file:
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@@
+      (effects (font (size 1.27 1.27)) hide)
+    )
+    (property "Digikey" "" (at 207.01 106.68 0)
+      (effects (font (size 1.27 1.27)) hide)
+    )
+    (property "MPN" "" (at 207.01 106.68 0)
+      (effects (font (size 1.27 1.27)) hide)
+    )
+    (property "Mouser" "" (at 207.01 106.68 0)
+      (effects (font (size 1.27 1.27)) hide)
+    )
+    (property "Field-1" "" (at 207.01 106.68 0)
       (effects (font (size 1.27 1.27)) hide)
     )
@@
     )
     (property "Quantity" "" (at 172.72 120.65 0)
+      (effects (font (size 1.27 1.27)) hide)
+    )
+    (property "Digikey" "" (at 172.72 120.65 0)
+      (effects (font (size 1.27 1.27)) hide)
+    )
+    (property "MPN" "" (at 172.72 120.65 0)
+      (effects (font (size 1.27 1.27)) hide)
+    )
+    (property "Mouser" "" (at 172.72 120.65 0)
+      (effects (font (size 1.27 1.27)) hide)
+    )
+    (property "Field-1" "" (at 172.72 120.65 0)
       (effects (font (size 1.27 1.27)) hide)
     )
@@
     )
     (property "Quantity" "" (at 132.08 110.49 0)
+      (effects (font (size 1.27 1.27)) hide)
+    )
+    (property "Digikey" "" (at 132.08 110.49 0)
+      (effects (font (size 1.27 1.27)) hide)
+    )
+    (property "MPN" "" (at 132.08 110.49 0)
+      (effects (font (size 1.27 1.27)) hide)
+    )
+    (property "Mouser" "" (at 132.08 110.49 0)
+      (effects (font (size 1.27 1.27)) hide)
+    )
+    (property "Field-1" "" (at 132.08 110.49 0)
       (effects (font (size 1.27 1.27)) hide)
     )
@@
       (effects (font (size 1.27 1.27)) hide)
     )
+    (property "Digikey" "" (at 118.11 87.63 0)
+      (effects (font (size 1.27 1.27)) hide)
+    )
+    (property "MPN" "GRM155R71H104KE14D " (at 118.11 87.63 0)
+      (effects (font (size 1.27 1.27)) hide)
+    )
+    (property "Mouser" "81-GRM155R71H104KE4D " (at 118.11 87.63 0)
+      (effects (font (size 1.27 1.27)) hide)
+    )
+    (property "Field-1" "" (at 118.11 87.63 0)
+      (effects (font (size 1.27 1.27)) hide)
+    )
+    (property "Manufacturer" "Murata" (at 118.11 87.63 0)
+      (effects (font (size 1.27 1.27)) hide)
+    )
+    (property "Voltage" "50V" (at 118.11 87.63 0)
+      (effects (font (size 1.27 1.27)) hide)
+    )
     (pin "1")
     (pin "2")
@@
     )
     (property "Quantity" "" (at 109.22 109.22 0)
+      (effects (font (size 1.27 1.27)) hide)
+    )
+    (property "Digikey" "" (at 109.22 109.22 0)
+      (effects (font (size 1.27 1.27)) hide)
+    )
+    (property "MPN" "" (at 109.22 109.22 0)
+      (effects (font (size 1.27 1.27)) hide)
+    )
+    (property "Mouser" "" (at 109.22 109.22 0)
+      (effects (font (size 1.27 1.27)) hide)
+    )
+    (property "Field-1" "" (at 109.22 109.22 0)
       (effects (font (size 1.27 1.27)) hide)
     )
@@
       (effects (font (size 1.27 1.27)) hide)
     )
+    (property "Digikey" "" (at 106.68 85.09 0)
+      (effects (font (size 1.27 1.27)) hide)
+    )
+    (property "MPN" "" (at 106.68 85.09 0)
+      (effects (font (size 1.27 1.27)) hide)
+    )
+    (property "Mouser" "" (at 106.68 85.09 0)
+      (effects (font (size 1.27 1.27)) hide)
+    )
+    (property "Field-1" "" (at 106.68 85.09 0)
+      (effects (font (size 1.27 1.27)) hide)
+    )
     (pin "1")
     (pin "2")
@@
       (effects (font (size 1.27 1.27)) hide)
     )
+    (property "Digikey" "" (at 158.75 78.74 0)
+      (effects (font (size 1.27 1.27)) hide)
+    )
+    (property "MPN" "" (at 158.75 78.74 0)
+      (effects (font (size 1.27 1.27)) hide)
+    )
+    (property "Mouser" "" (at 158.75 78.74 0)
+      (effects (font (size 1.27 1.27)) hide)
+    )
+    (property "Field-1" "" (at 158.75 78.74 0)
+      (effects (font (size 1.27 1.27)) hide)
+    )

Commit message: Oops, hadn't run the ERC for ages. Ran, passed. Add ERC and DRC exclusions where unavoidable
Parts:
- J15: Digikey (none) -> 609-4618-6-ND; MPN (none) -> 10118194-0001LF; Manufacturer (none) -> Amphenol; Mouser (none) -> 649-10118194-0001LF
- Q4: Digikey (none) -> 1727-1280-6-ND; MPN (none) -> NX3008NBKW; Manufacturer (none) -> Nexperia; Mouser (none) -> 771-NX3008NBKW,115
- U15: Digikey (none) -> FSUSB42MUXDKR-ND; MPN (none) -> FSUSB42MUX; Manufacturer (none) -> On Semi; Mouser (none) -> 512-FSUSB42MUX
- U16: Digikey (none) -> ESD7004MUTAGOSDKR-ND; MPN (none) -> ESD7004MUTAG; Manufacturer (none) -> On Semi; Mouser (none) -> 863-ESD7004MUTAG
Changed lines of the file:
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@@
-      (effects (font (size 1.27 1.27)) hide)
-    )
-    (property "MANUFACTURER" "" (at 207.01 106.68 0)
       (effects (font (size 1.27 1.27)) hide)
     )
@@
       (effects (font (size 1.27 1.27)) hide)
     )
-    (property "Digikey" "" (at 207.01 106.68 0)
-      (effects (font (size 1.27 1.27)) hide)
-    )
-    (property "MPN" "" (at 207.01 106.68 0)
-      (effects (font (size 1.27 1.27)) hide)
-    )
-    (property "Mouser" "" (at 207.01 106.68 0)
+    (property "Digikey" "609-4618-6-ND" (at 207.01 106.68 0)
+      (effects (font (size 1.27 1.27)) hide)
+    )
+    (property "MPN" "10118194-0001LF" (at 207.01 106.68 0)
+      (effects (font (size 1.27 1.27)) hide)
+    )
+    (property "Mouser" "649-10118194-0001LF" (at 207.01 106.68 0)
+      (effects (font (size 1.27 1.27)) hide)
+    )
+    (property "Manufacturer" "Amphenol" (at 207.01 106.68 0)
+      (effects (font (size 1.27 1.27)) hide)
+    )
+    (property "Farnell" "" (at 207.01 106.68 0)
       (effects (font (size 1.27 1.27)) hide)
     )
@@
       (effects (font (size 1.27 1.27)) hide)
     )
-    (property "MANUFACTURER" "" (at 172.72 120.65 0)
-      (effects (font (size 1.27 1.27)) hide)
-    )
     (property "Quantity" "" (at 172.72 120.65 0)
       (effects (font (size 1.27 1.27)) hide)
     )
-    (property "Digikey" "" (at 172.72 120.65 0)
-      (effects (font (size 1.27 1.27)) hide)
-    )
-    (property "MPN" "" (at 172.72 120.65 0)
-      (effects (font (size 1.27 1.27)) hide)
-    )
-    (property "Mouser" "" (at 172.72 120.65 0)
+    (property "Digikey" "ESD7004MUTAGOSDKR-ND" (at 172.72 120.65 0)
+      (effects (font (size 1.27 1.27)) hide)
+    )
+    (property "MPN" "ESD7004MUTAG" (at 172.72 120.65 0)
+      (effects (font (size 1.27 1.27)) hide)
+    )
+    (property "Mouser" "863-ESD7004MUTAG" (at 172.72 120.65 0)
+      (effects (font (size 1.27 1.27)) hide)
+    )
+    (property "Farnell" "" (at 172.72 120.65 0)
       (effects (font (size 1.27 1.27)) hide)
     )
     (property "Field-1" "" (at 172.72 120.65 0)
+      (effects (font (size 1.27 1.27)) hide)
+    )
+    (property "Manufacturer" "On Semi" (at 172.72 120.65 0)
       (effects (font (size 1.27 1.27)) hide)
     )
@@
       (effects (font (size 1.27 1.27)) hide)
     )
-    (property "MANUFACTURER" "" (at 132.08 110.49 0)
-      (effects (font (size 1.27 1.27)) hide)
-    )
     (property "Quantity" "" (at 132.08 110.49 0)
       (effects (font (size 1.27 1.27)) hide)
     )
-    (property "Digikey" "" (at 132.08 110.49 0)
-      (effects (font (size 1.27 1.27)) hide)
-    )
-    (property "MPN" "" (at 132.08 110.49 0)
-      (effects (font (size 1.27 1.27)) hide)
-    )
-    (property "Mouser" "" (at 132.08 110.49 0)
+    (property "Digikey" "FSUSB42MUXDKR-ND" (at 132.08 110.49 0)
+      (effects (font (size 1.27 1.27)) hide)
+    )
+    (property "MPN" "FSUSB42MUX" (at 132.08 110.49 0)
+      (effects (font (size 1.27 1.27)) hide)
+    )
+    (property "Mouser" "512-FSUSB42MUX" (at 132.08 110.49 0)
+      (effects (font (size 1.27 1.27)) hide)
+    )
+    (property "Farnell" "" (at 132.08 110.49 0)
       (effects (font (size 1.27 1.27)) hide)
     )
     (property "Field-1" "" (at 132.08 110.49 0)
+      (effects (font (size 1.27 1.27)) hide)
+    )
+    (property "Manufacturer" "On Semi" (at 132.08 110.49 0)
       (effects (font (size 1.27 1.27)) hide)
     )
@@
       (effects (font (size 1.27 1.27)) hide)
     )
-    (property "MANUFACTURER" "" (at 118.11 87.63 0)
-      (effects (font (size 1.27 1.27)) hide)
-    )
     (property "Quantity" "" (at 118.11 87.63 0)
       (effects (font (size 1.27 1.27)) hide)
@@
       (effects (font (size 1.27 1.27)) hide)
     )
+    (property "Manufacturer" "Murata" (at 118.11 87.63 0)
+      (effects (font (size 1.27 1.27)) hide)
+    )
+    (property "Voltage" "50V" (at 118.11 87.63 0)
+      (effects (font (size 1.27 1.27)) hide)
+    )
+    (property "Farnell" "" (at 118.11 87.63 0)
+      (effects (font (size 1.27 1.27)) hide)
+    )
     (property "Field-1" "" (at 118.11 87.63 0)
-      (effects (font (size 1.27 1.27)) hide)
-    )
-    (property "Manufacturer" "Murata" (at 118.11 87.63 0)
-      (effects (font (size 1.27 1.27)) hide)
-    )
-    (property "Voltage" "50V" (at 118.11 87.63 0)
       (effects (font (size 1.27 1.27)) hide)
     )
@@
       (effects (font (size 1.27 1.27)) hide)
     )
-    (property "MANUFACTURER" "" (at 109.22 109.22 0)
-      (effects (font (size 1.27 1.27)) hide)
-    )
     (property "Quantity" "" (at 109.22 109.22 0)
       (effects (font (size 1.27 1.27)) hide)
@@
     )
     (property "Mouser" "" (at 109.22 109.22 0)
+      (effects (font (size 1.27 1.27)) hide)
+    )
+    (property "Farnell" "" (at 109.22 109.22 0)
       (effects (font (size 1.27 1.27)) hide)
     )
@@
       (effects (font (size 1.27 1.27)) hide)
     )
-    (property "MANUFACTURER" "" (at 106.68 85.09 0)
-      (effects (font (size 1.27 1.27)) hide)
-    )
     (property "Quantity" "" (at 106.68 85.09 0)
       (effects (font (size 1.27 1.27)) hide)
@@
     )
     (property "Mouser" "" (at 106.68 85.09 0)
+      (effects (font (size 1.27 1.27)) hide)
+    )
+    (property "Farnell" "" (at 106.68 85.09 0)
       (effects (font (size 1.27 1.27)) hide)
     )
@@
       (effects (font (size 1.27 1.27)) hide)
     )
-    (property "MANUFACTURER" "" (at 158.75 78.74 0)
-      (effects (font (size 1.27 1.27)) hide)
-    )
     (property "Quantity" "" (at 158.75 78.74 0)
       (effects (font (size 1.27 1.27)) hide)
     )
-    (property "Digikey" "" (at 158.75 78.74 0)
-      (effects (font (size 1.27 1.27)) hide)
-    )
-    (property "MPN" "" (at 158.75 78.74 0)
-      (effects (font (size 1.27 1.27)) hide)
-    )
-    (property "Mouser" "" (at 158.75 78.74 0)
+    (property "Digikey" "1727-1280-6-ND" (at 158.75 78.74 0)
+      (effects (font (size 1.27 1.27)) hide)
+    )
+    (property "MPN" "NX3008NBKW" (at 158.75 78.74 0)
+      (effects (font (size 1.27 1.27)) hide)
+    )
+    (property "Mouser" "771-NX3008NBKW,115" (at 158.75 78.74 0)
+      (effects (font (size 1.27 1.27)) hide)
+    )
+    (property "Farnell" "" (at 158.75 78.74 0)
       (effects (font (size 1.27 1.27)) hide)
     )
@@
       (effects (font (size 1.27 1.27)) hide)
     )
+    (property "Manufacturer" "Nexperia" (at 158.75 78.74 0)
+      (effects (font (size 1.27 1.27)) hide)
+    )
