File: r5/src/_external_mic.kicad_sch (KiCad schematic)
At the start: 139 parts, among them Q12 BSS84PW, Q13 BSS84PW, Q14 NX6008NBKW, Q15 NX3008NBKW, Q16 NX3008NBKW, Q17 NX3008NBKW, Q18 NX3008NBKW, Q19 NX3008NBKW, Q20 BSS84PW, Q21 BSS84PW, Q22 NX3008NBKW, Q23 NX3008NBKW, Q24 NX3008NBKW, Q25 Si2323DS, Q29 Si2323DS, Q30 NX3008NBKW, T18 , T19 , T20 , T23 , T24 , T25 , T26 , T27 , T28 , T29 , T30 , T31 , T32 , T33 , T34 , T35 , T37 , T38 , T43 , T44 , T45 , T46 , T47 , T48 , T49 , T50 , T59 , U17 74HC20, U18 THAT5173, U19 74HC74, U20 74HC132, U21 74HC4520, U22 74HC132, U23 THAT1580, U24 74HC688, U25 LM4562, U26 74HC688, U27 AD4005, U36 APX809S-40SA

Commit message: Oops, hadn't run the ERC for ages. Ran, passed. Add ERC and DRC exclusions where unavoidable
Parts:
- C27, C46: Tempco (none) -> NP0
- C49, C50: MPN (none) -> EMVH630ADA470MHA0G; Manufacturer (none) -> United Chemi-Con; Mouser (none) -> 565-4268-1-ND
- C71: Voltage (none) -> 100V
- C77, C83, C84: MPN (none) -> CL10A106MQ8NNNC; Manufacturer (none) -> Samsung; Mouser (none) -> 187-CL10A106MQ8NNNC
- D10, D11, D12, D13, D14, D8: Digikey (none) -> 1727-1347-1-ND; MPN (none) -> PMEG6020ETR,115; Manufacturer (none) -> Nexperia
- D15: Digikey (none) -> BZT52C1213-FDIDKR-ND; MPN (none) -> BZT52C12-13-F; Manufacturer (none) -> Diodes Inc.; Mouser (none) -> 621-BZT52C12-13-F
- D26, D27: MPN (none) -> 1SS387,L3F; Manufacturer (none) -> Toshiba; Mouser (none) -> 757-1SS387L3F
- FB3: Digikey (none) -> 490-17349-1-ND; MPN (none) -> BLM18KG102SN1D; Manufacturer (none) -> Murata
- Q12, Q13, Q20, Q21: MPN (none) -> BSS84PW; Manufacturer (none) -> Infineon; Mouser (none) -> 726-BSS84PWH6327XTSA
- Q14: value NX6008NBKW -> NX3008NBKW; Digikey (none) -> 1727-1280-6-ND; MPN (none) -> NX3008NBKW; Manufacturer (none) -> Nexperia; Mouser (none) -> 771-NX3008NBKW,115
- Q15, Q16, Q17, Q18, Q19, Q22, Q23, Q24, Q30: Digikey (none) -> 1727-1280-6-ND; MPN (none) -> NX3008NBKW; Manufacturer (none) -> Nexperia; Mouser (none) -> 771-NX3008NBKW,115
- Q25, Q29: MPN (none) -> SI2323DS-T1; Manufacturer (none) -> Vishay
- R47: Tolerance (none) -> 0.1%
- R48: Tolerance 0.1% thin film -> 0.1%
- R51, R52: MPN (none) -> ERA-2AEB122X; Manufacturer (none) -> Panasonic; Mouser (none) -> 667-ERA-2AEB122X
- R53, R54, R57, R60: MPN (none) -> ERA-2AEB102X; Manufacturer (none) -> Panasonic; Mouser (none) -> 667-ERA-2AEB102X
- R55, R56, R58, R59: MPN (none) -> ERA-2AEB822X; Manufacturer (none) -> Panasonic; Mouser (none) -> 667-ERA-2AEB822X
- R61, R62: MPN (none) -> ERA-2AEB201X; Manufacturer (none) -> Panasonic; Mouser (none) -> 667-ERA-2AEB201X
- U17: MPN (none) -> 74HC20PW; Manufacturer (none) -> Nexperia; Mouser (none) -> 771-HC20PW118
- U18: MPN (none) -> 5173N24-U; Manufacturer (none) -> THAT Corp; Mouser (none) -> 887-5173N24-U
- U19: MPN (none) -> 74HC74PW; Manufacturer (none) -> Nexperia; Mouser (none) -> 771-74HC74PW-T
- U20, U22: MPN (none) -> 74HC132PW; Manufacturer (none) -> Nexperia; Mouser (none) -> 771-74HC132PW-T
- U21: MPN (none) -> 74HC4520PW; Manufacturer (none) -> Nexperia; Mouser (none) -> 771-HC4520PW118
- U23: MPN (none) -> 1580N16-U; Manufacturer (none) -> THAT Corp; Mouser (none) -> 887-1580N16-U
- U24, U26: MPN (none) -> 74HC688PW; Manufacturer (none) -> Nexperia; Mouser (none) -> 771-HC688PW118
- U25: MPN (none) -> LM4562MA; Manufacturer (none) -> TI; Mouser (none) -> 926-LM4562MAX/NOPB
- U27: MPN (none) -> AD4005BRMZ; Manufacturer (none) -> Analog; Mouser (none) -> 584-AD4005BRMZ

Commit message: Exclude all testpoints from BoM. Correct some BoM errors
Parts:
- T18, T19, T20, T23, T24, T25, T26, T27, T28, T29, T30, T31, T34, T35, T37, T38, T43, T44, T45, T46, T47, T48, T49, T50, T59: now left out of the parts list
- U36: MPN (none) -> APX809S-40SA; Manufacturer (none) -> Diodes Inc.; Mouser (none) -> 621-APX809S-40SA-7
