File: r5/src/_rtc.kicad_sch (KiCad schematic)
At the start: 9 parts, among them U13 DS3231MZ, U14 74LVC1G07DCK

Commit message: Update schematic to include the latest library symbols. Mainly this updated the symbol fields, but three symbols actually changed, which required schematic edits to reconnect their pins. No circuit changes were made, and this was verified by checking the preview data in the PCB's "Update PCB from Schematic..." dialog.
Connections:
- no-connect marks 2 -> 3
Changed lines of the file:
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@@
   (junction (at 151.13 99.06) (diameter 1.016) (color 0 0 0 0)
   )
-  (junction (at 168.91 99.06) (diameter 1.016) (color 0 0 0 0)
-  )
-  (junction (at 185.42 83.82) (diameter 1.016) (color 0 0 0 0)
+  (junction (at 180.34 83.82) (diameter 0) (color 0 0 0 0)
   )
   (junction (at 106.68 72.39) (diameter 1.016) (color 0 0 0 0)
   )
+  (junction (at 168.91 99.06) (diameter 0) (color 0 0 0 0)
+  )
   (junction (at 93.98 72.39) (diameter 0) (color 0 0 0 0)
   )
@@
   )
   (no_connect (at 135.89 91.44))
+  (no_connect (at 182.88 109.22))
   (no_connect (at 110.49 101.6))
   (wire (pts (xy 168.91 83.82) (xy 168.91 88.9))
     (stroke (width 0) (type solid))
   )
-  (wire (pts (xy 185.42 76.2) (xy 185.42 83.82))
+  (wire (pts (xy 180.34 78.74) (xy 180.34 83.82))
     (stroke (width 0) (type solid))
   )
@@
   )
   (wire (pts (xy 163.83 99.06) (xy 168.91 99.06))
-    (stroke (width 0) (type solid))
-  )
-  (wire (pts (xy 168.91 99.06) (xy 177.8 99.06))
     (stroke (width 0) (type solid))
   )
@@
     (stroke (width 0) (type solid))
   )
-  (wire (pts (xy 168.91 83.82) (xy 185.42 83.82))
-    (stroke (width 0) (type solid))
-  )
-  (wire (pts (xy 185.42 83.82) (xy 185.42 96.52))
-    (stroke (width 0) (type solid))
-  )
-  (wire (pts (xy 185.42 101.6) (xy 185.42 107.95))
-    (stroke (width 0) (type solid))
+  (wire (pts (xy 168.91 83.82) (xy 180.34 83.82))
+    (stroke (width 0) (type solid))
+  )
+  (wire (pts (xy 180.34 83.82) (xy 180.34 88.9))
+    (stroke (width 0) (type solid))
+  )
+  (wire (pts (xy 198.12 99.06) (xy 200.66 99.06))
+    (stroke (width 0) (type default))
   )
   (wire (pts (xy 123.19 72.39) (xy 128.27 72.39))
@@
   )
   (wire (pts (xy 168.91 93.98) (xy 168.91 99.06))
+    (stroke (width 0) (type solid))
+  )
+  (wire (pts (xy 168.91 99.06) (xy 170.18 99.06))
     (stroke (width 0) (type solid))
   )
@@
   )
   (wire (pts (xy 128.27 81.28) (xy 128.27 80.01))
-    (stroke (width 0) (type solid))
-  )
-  (wire (pts (xy 191.77 99.06) (xy 200.66 99.06))
     (stroke (width 0) (type solid))
   )
@@
     )
   )
-  (symbol (lib_id "power:+5V") (at 185.42 76.2 0) (unit 1)
-    (exclude_from_sim no) (in_bom yes) (on_board yes) (dnp no)
-    (property "Reference" "#PWR0177" (at 185.42 80.01 0)
-      (effects (font (size 1.27 1.27)) hide)
-    )
-    (property "Value" "+5V" (at 186.69 71.12 0)
-      (effects (font (size 1.27 1.27)))
-    )
-    (property "Footprint" "" (at 185.42 76.2 0)
-      (effects (font (size 1.27 1.27)) hide)
-    )
-    (property "Datasheet" "" (at 185.42 76.2 0)
-      (effects (font (size 1.27 1.27)) hide)
-    )
-    (property "Description" "" (at 185.42 76.2 0)
+  (symbol (lib_id "power:+5V") (at 180.34 78.74 0) (unit 1)
+    (exclude_from_sim no) (in_bom yes) (on_board yes) (dnp no)
+    (property "Reference" "#PWR0177" (at 180.34 82.55 0)
+      (effects (font (size 1.27 1.27)) hide)
+    )
+    (property "Value" "+5V" (at 181.61 73.66 0)
+      (effects (font (size 1.27 1.27)))
+    )
+    (property "Footprint" "" (at 180.34 78.74 0)
+      (effects (font (size 1.27 1.27)) hide)
+    )
+    (property "Datasheet" "" (at 180.34 78.74 0)
+      (effects (font (size 1.27 1.27)) hide)
+    )
+    (property "Description" "" (at 180.34 78.74 0)
       (effects (font (size 1.27 1.27)) hide)
     )
@@
     )
   )
-  (symbol (lib_id "power:GND") (at 185.42 107.95 0) (unit 1)
-    (exclude_from_sim no) (in_bom yes) (on_board yes) (dnp no)
-    (property "Reference" "#PWR0178" (at 185.42 114.3 0)
-      (effects (font (size 1.27 1.27)) hide)
-    )
-    (property "Value" "GND" (at 186.69 113.03 0)
-      (effects (font (size 1.27 1.27)))
-    )
-    (property "Footprint" "" (at 185.42 107.95 0)
-      (effects (font (size 1.27 1.27)) hide)
-    )
-    (property "Datasheet" "" (at 185.42 107.95 0)
-      (effects (font (size 1.27 1.27)) hide)
-    )
-    (property "Description" "" (at 185.42 107.95 0)
+  (symbol (lib_id "power:GND") (at 180.34 109.22 0) (unit 1)
+    (exclude_from_sim no) (in_bom yes) (on_board yes) (dnp no) (fields_autoplaced)
+    (property "Reference" "#PWR0178" (at 180.34 115.57 0)
+      (effects (font (size 1.27 1.27)) hide)
+    )
+    (property "Value" "GND" (at 180.34 114.3 0)
+      (effects (font (size 1.27 1.27)))
+    )
+    (property "Footprint" "" (at 180.34 109.22 0)
+      (effects (font (size 1.27 1.27)) hide)
+    )
+    (property "Datasheet" "" (at 180.34 109.22 0)
+      (effects (font (size 1.27 1.27)) hide)
+    )
+    (property "Description" "" (at 180.34 109.22 0)
       (effects (font (size 1.27 1.27)) hide)
     )
@@
     (pin "4")
     (pin "5")
-    (instances
-      (project "bugg-main-r5"
+    (pin "1")
+    (instances
+      (project "bugg-main-r5"

Commit message: Update layout to standardise on 0402 passives everywhere possible. This reduces the number of BoM lines. DRC passed. Add DRC exclusions for unavoidable violations
Parts:
- C34, C35, C36: footprint Capacitor_SMD:C_0603_1608Metric -> Capacitor_SMD:C_0402_1005Metric
- R29, R30: footprint Resistor_SMD:R_0603_1608Metric -> Resistor_SMD:R_0402_1005Metric
Changed lines of the file:
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@@
       (effects (font (size 1.27 1.27)) (justify left))
     )
-    (property "Footprint" "Capacitor_SMD:C_0603_1608Metric" (at 128.27 77.47 0)
+    (property "Footprint" "Capacitor_SMD:C_0402_1005Metric" (at 128.27 77.47 0)
       (effects (font (size 1.27 1.27)) hide)
     )
@@
       (effects (font (size 1.27 1.27)))
     )
-    (property "Footprint" "Capacitor_SMD:C_0603_1608Metric" (at 161.29 99.06 0)
+    (property "Footprint" "Capacitor_SMD:C_0402_1005Metric" (at 161.29 99.06 0)
       (effects (font (size 1.27 1.27)) hide)
     )
@@
       (effects (font (size 1.27 1.27)) (justify right))
     )
-    (property "Footprint" "Resistor_SMD:R_0603_1608Metric" (at 168.91 91.44 0)
+    (property "Footprint" "Resistor_SMD:R_0402_1005Metric" (at 168.91 91.44 0)
       (effects (font (size 1.27 1.27)) hide)
     )
@@
       (effects (font (size 1.27 1.27)) (justify right))
     )
-    (property "Footprint" "Resistor_SMD:R_0603_1608Metric" (at 151.13 91.44 0)
+    (property "Footprint" "Resistor_SMD:R_0402_1005Metric" (at 151.13 91.44 0)
       (effects (font (size 1.27 1.27)) hide)
     )
@@
       (effects (font (size 1.27 1.27)) (justify left))
     )
-    (property "Footprint" "Capacitor_SMD:C_0603_1608Metric" (at 93.98 77.47 0)
-      (effects (font (size 1.27 1.27)) hide)
-    )
+    (property "Footprint" "Capacitor_SMD:C_0402_1005Metric" (at 93.98 77.47 0)
+      (effects (font (size 1.27 1.27)) hide)
+    )

Commit message: Change 0805 47uF to 1206 to save a BOM line. Update layout, DRC pass.
Parts:
- BT1: Digikey (none) -> 36-3000CT-ND; MPN (none) -> 3000TR; Manufacturer (none) -> Keystone; Mouser (none) -> 534-3000TR
- C34, C35, C36: MPN (none) -> GRM155R71H104KE14D; Manufacturer (none) -> Murata; Mouser (none) -> 81-GRM155R71H104KE4D; Voltage (none) -> 50V
Changed lines of the file:
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@@
+      (effects (font (size 1.27 1.27)) hide)
+    )
+    (property "Digikey" "" (at 82.55 77.47 0)
+      (effects (font (size 1.27 1.27)) hide)
+    )
+    (property "MPN" "" (at 82.55 77.47 0)
+      (effects (font (size 1.27 1.27)) hide)
+    )
+    (property "Mouser" "" (at 82.55 77.47 0)
+      (effects (font (size 1.27 1.27)) hide)
+    )
+    (property "Field-1" "" (at 82.55 77.47 0)
       (effects (font (size 1.27 1.27)) hide)
     )
@@
       (effects (font (size 1.27 1.27)) hide)
     )
+    (property "Digikey" "" (at 128.27 77.47 0)
+      (effects (font (size 1.27 1.27)) hide)
+    )
+    (property "MPN" "GRM155R71H104KE14D " (at 128.27 77.47 0)
+      (effects (font (size 1.27 1.27)) hide)
+    )
+    (property "Mouser" "81-GRM155R71H104KE4D " (at 128.27 77.47 0)
+      (effects (font (size 1.27 1.27)) hide)
+    )
+    (property "Field-1" "" (at 128.27 77.47 0)
+      (effects (font (size 1.27 1.27)) hide)
+    )
+    (property "Manufacturer" "Murata" (at 128.27 77.47 0)
+      (effects (font (size 1.27 1.27)) hide)
+    )
+    (property "Voltage" "50V" (at 128.27 77.47 0)
+      (effects (font (size 1.27 1.27)) hide)
+    )
     (pin "1")
     (pin "2")
@@
     )
     (property "Quantity" "" (at 185.42 99.06 0)
+      (effects (font (size 1.27 1.27)) hide)
+    )
+    (property "Digikey" "" (at 185.42 99.06 0)
+      (effects (font (size 1.27 1.27)) hide)
+    )
+    (property "MPN" "" (at 185.42 99.06 0)
+      (effects (font (size 1.27 1.27)) hide)
+    )
+    (property "Mouser" "" (at 185.42 99.06 0)
+      (effects (font (size 1.27 1.27)) hide)
+    )
+    (property "Field-1" "" (at 185.42 99.06 0)
       (effects (font (size 1.27 1.27)) hide)
     )
@@
       (effects (font (size 1.27 1.27)) hide)
     )
+    (property "Digikey" "36-3000CT-ND" (at 106.68 78.74 0)
+      (effects (font (size 1.27 1.27)) hide)
+    )
+    (property "MPN" "3000TR" (at 106.68 78.74 0)
+      (effects (font (size 1.27 1.27)) hide)
+    )
+    (property "Manufacturer" "Keystone" (at 106.68 78.74 0)
+      (effects (font (size 1.27 1.27)) hide)
+    )
+    (property "Mouser" "534-3000TR" (at 106.68 78.74 0)
+      (effects (font (size 1.27 1.27)) hide)
+    )
+    (property "Field-1" "" (at 106.68 78.74 0)
+      (effects (font (size 1.27 1.27)) hide)
+    )
     (pin "1")
     (pin "2")
@@
     )
     (property "Quantity" "" (at 161.29 99.06 0)
+      (effects (font (size 1.27 1.27)) hide)
+    )
+    (property "Digikey" "" (at 161.29 99.06 0)
+      (effects (font (size 1.27 1.27)) hide)
+    )
+    (property "MPN" "GRM155R71H104KE14D " (at 161.29 99.06 0)
+      (effects (font (size 1.27 1.27)) hide)
+    )
+    (property "Mouser" "81-GRM155R71H104KE4D " (at 161.29 99.06 0)
+      (effects (font (size 1.27 1.27)) hide)
+    )
+    (property "Field-1" "" (at 161.29 99.06 0)
+      (effects (font (size 1.27 1.27)) hide)
+    )
+    (property "Manufacturer" "Murata" (at 161.29 99.06 0)
+      (effects (font (size 1.27 1.27)) hide)
+    )
+    (property "Voltage" "50V" (at 161.29 99.06 0)
       (effects (font (size 1.27 1.27)) hide)
     )
@@
       (effects (font (size 1.27 1.27)) hide)
     )
+    (property "Digikey" "" (at 168.91 91.44 0)
+      (effects (font (size 1.27 1.27)) hide)
+    )
+    (property "MPN" "" (at 168.91 91.44 0)
+      (effects (font (size 1.27 1.27)) hide)
+    )
+    (property "Mouser" "" (at 168.91 91.44 0)
+      (effects (font (size 1.27 1.27)) hide)
+    )
+    (property "Field-1" "" (at 168.91 91.44 0)
+      (effects (font (size 1.27 1.27)) hide)
+    )
     (pin "1")
     (pin "2")
@@
       (effects (font (size 1.27 1.27)) hide)
     )
+    (property "Digikey" "" (at 151.13 91.44 0)
+      (effects (font (size 1.27 1.27)) hide)
+    )
+    (property "MPN" "" (at 151.13 91.44 0)
+      (effects (font (size 1.27 1.27)) hide)
+    )
+    (property "Mouser" "" (at 151.13 91.44 0)
+      (effects (font (size 1.27 1.27)) hide)
+    )
+    (property "Field-1" "" (at 151.13 91.44 0)
+      (effects (font (size 1.27 1.27)) hide)
+    )
     (pin "1")
     (pin "2")
@@
     )
     (property "Quantity" "" (at 123.19 96.52 0)
+      (effects (font (size 1.27 1.27)) hide)
+    )
+    (property "Digikey" "" (at 123.19 96.52 0)
+      (effects (font (size 1.27 1.27)) hide)
+    )
+    (property "MPN" "" (at 123.19 96.52 0)
+      (effects (font (size 1.27 1.27)) hide)
+    )
+    (property "Mouser" "" (at 123.19 96.52 0)
+      (effects (font (size 1.27 1.27)) hide)
+    )
+    (property "Field-1" "" (at 123.19 96.52 0)
       (effects (font (size 1.27 1.27)) hide)
     )
@@
       (effects (font (size 1.27 1.27)) hide)
     )
+    (property "Digikey" "" (at 93.98 77.47 0)
+      (effects (font (size 1.27 1.27)) hide)
+    )
+    (property "MPN" "GRM155R71H104KE14D " (at 93.98 77.47 0)
+      (effects (font (size 1.27 1.27)) hide)
+    )
+    (property "Mouser" "81-GRM155R71H104KE4D " (at 93.98 77.47 0)
+      (effects (font (size 1.27 1.27)) hide)
+    )
+    (property "Field-1" "" (at 93.98 77.47 0)
+      (effects (font (size 1.27 1.27)) hide)
+    )
+    (property "Manufacturer" "Murata" (at 93.98 77.47 0)
+      (effects (font (size 1.27 1.27)) hide)
+    )
+    (property "Voltage" "50V" (at 93.98 77.47 0)
+      (effects (font (size 1.27 1.27)) hide)
+    )

Commit message: Oops, hadn't run the ERC for ages. Ran, passed. Add ERC and DRC exclusions where unavoidable
Parts:
- D20: Digikey (none) -> 283-2964-6-ND; MPN (none) -> 0402ESDA-MLP1; Manufacturer (none) -> Eaton; Mouser (none) -> 504-0402ESDA-MLP1
- U13: Digikey (none) -> DS3231MZ+-ND; MPN (none) -> DS3231MZ+; Manufacturer (none) -> Maxim; Mouser (none) -> 700-DS3231MZ+
- U14: Digikey (none) -> 296-26591-6-ND; MPN (none) -> SN74LVC1G07DCKT; Manufacturer (none) -> TI; Mouser (none) -> 595-SN74LVC1G07DCK3
Changed lines of the file:
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@@
-      (effects (font (size 1.27 1.27)) hide)
-    )
-    (property "MANUFACTURER" "" (at 82.55 77.47 0)
       (effects (font (size 1.27 1.27)) hide)
     )
@@
       (effects (font (size 1.27 1.27)) hide)
     )
-    (property "Digikey" "" (at 82.55 77.47 0)
-      (effects (font (size 1.27 1.27)) hide)
-    )
-    (property "MPN" "" (at 82.55 77.47 0)
-      (effects (font (size 1.27 1.27)) hide)
-    )
-    (property "Mouser" "" (at 82.55 77.47 0)
+    (property "Digikey" "283-2964-6-ND" (at 82.55 77.47 0)
+      (effects (font (size 1.27 1.27)) hide)
+    )
+    (property "MPN" "0402ESDA-MLP1" (at 82.55 77.47 0)
+      (effects (font (size 1.27 1.27)) hide)
+    )
+    (property "Mouser" "504-0402ESDA-MLP1" (at 82.55 77.47 0)
+      (effects (font (size 1.27 1.27)) hide)
+    )
+    (property "Manufacturer" "Eaton" (at 82.55 77.47 0)
+      (effects (font (size 1.27 1.27)) hide)
+    )
+    (property "Farnell" "" (at 82.55 77.47 0)
       (effects (font (size 1.27 1.27)) hide)
     )
@@
       (effects (font (size 1.27 1.27)) hide)
     )
-    (property "MANUFACTURER" "" (at 128.27 77.47 0)
-      (effects (font (size 1.27 1.27)) hide)
-    )
     (property "Quantity" "" (at 128.27 77.47 0)
       (effects (font (size 1.27 1.27)) hide)
@@
       (effects (font (size 1.27 1.27)) hide)
     )
+    (property "Manufacturer" "Murata" (at 128.27 77.47 0)
+      (effects (font (size 1.27 1.27)) hide)
+    )
+    (property "Voltage" "50V" (at 128.27 77.47 0)
+      (effects (font (size 1.27 1.27)) hide)
+    )
+    (property "Farnell" "" (at 128.27 77.47 0)
+      (effects (font (size 1.27 1.27)) hide)
+    )
     (property "Field-1" "" (at 128.27 77.47 0)
       (effects (font (size 1.27 1.27)) hide)
     )
-    (property "Manufacturer" "Murata" (at 128.27 77.47 0)
-      (effects (font (size 1.27 1.27)) hide)
-    )
-    (property "Voltage" "50V" (at 128.27 77.47 0)
-      (effects (font (size 1.27 1.27)) hide)
-    )
     (pin "1")
     (pin "2")
@@
       (effects (font (size 1.27 1.27)) hide)
     )
-    (property "MANUFACTURER" "" (at 185.42 99.06 0)
-      (effects (font (size 1.27 1.27)) hide)
-    )
     (property "Quantity" "" (at 185.42 99.06 0)
       (effects (font (size 1.27 1.27)) hide)
     )
-    (property "Digikey" "" (at 185.42 99.06 0)
-      (effects (font (size 1.27 1.27)) hide)
-    )
-    (property "MPN" "" (at 185.42 99.06 0)
-      (effects (font (size 1.27 1.27)) hide)
-    )
-    (property "Mouser" "" (at 185.42 99.06 0)
+    (property "Digikey" "296-26591-6-ND" (at 185.42 99.06 0)
+      (effects (font (size 1.27 1.27)) hide)
+    )
+    (property "MPN" "SN74LVC1G07DCKT" (at 185.42 99.06 0)
+      (effects (font (size 1.27 1.27)) hide)
+    )
+    (property "Mouser" "595-SN74LVC1G07DCK3" (at 185.42 99.06 0)
+      (effects (font (size 1.27 1.27)) hide)
+    )
+    (property "Farnell" "" (at 185.42 99.06 0)
       (effects (font (size 1.27 1.27)) hide)
     )
     (property "Field-1" "" (at 185.42 99.06 0)
+      (effects (font (size 1.27 1.27)) hide)
+    )
+    (property "Manufacturer" "TI" (at 185.42 99.06 0)
       (effects (font (size 1.27 1.27)) hide)
     )
@@
       (effects (font (size 1.27 1.27)) hide)
     )
-    (property "MANUFACTURER" "" (at 106.68 78.74 0)
-      (effects (font (size 1.27 1.27)) hide)
-    )
     (property "Quantity" "" (at 106.68 78.74 0)
       (effects (font (size 1.27 1.27)) hide)
@@
       (effects (font (size 1.27 1.27)) hide)
     )
+    (property "Farnell" "" (at 106.68 78.74 0)
+      (effects (font (size 1.27 1.27)) hide)
+    )
     (property "Field-1" "" (at 106.68 78.74 0)
       (effects (font (size 1.27 1.27)) hide)
@@
       (effects (font (size 1.27 1.27)) hide)
     )
-    (property "MANUFACTURER" "" (at 161.29 99.06 0)
-      (effects (font (size 1.27 1.27)) hide)
-    )
     (property "Quantity" "" (at 161.29 99.06 0)
       (effects (font (size 1.27 1.27)) hide)
@@
       (effects (font (size 1.27 1.27)) hide)
     )
+    (property "Manufacturer" "Murata" (at 161.29 99.06 0)
+      (effects (font (size 1.27 1.27)) hide)
+    )
+    (property "Voltage" "50V" (at 161.29 99.06 0)
+      (effects (font (size 1.27 1.27)) hide)
+    )
+    (property "Farnell" "" (at 161.29 99.06 0)
+      (effects (font (size 1.27 1.27)) hide)
+    )
     (property "Field-1" "" (at 161.29 99.06 0)
-      (effects (font (size 1.27 1.27)) hide)
-    )
-    (property "Manufacturer" "Murata" (at 161.29 99.06 0)
-      (effects (font (size 1.27 1.27)) hide)
-    )
-    (property "Voltage" "50V" (at 161.29 99.06 0)
       (effects (font (size 1.27 1.27)) hide)
     )
@@
       (effects (font (size 1.27 1.27)) hide)
     )
-    (property "MANUFACTURER" "" (at 168.91 91.44 0)
-      (effects (font (size 1.27 1.27)) hide)
-    )
     (property "Quantity" "" (at 168.91 91.44 0)
       (effects (font (size 1.27 1.27)) hide)
@@
     )
     (property "Mouser" "" (at 168.91 91.44 0)
+      (effects (font (size 1.27 1.27)) hide)
+    )
+    (property "Farnell" "" (at 168.91 91.44 0)
       (effects (font (size 1.27 1.27)) hide)
     )
@@
       (effects (font (size 1.27 1.27)) hide)
     )
-    (property "MANUFACTURER" "" (at 151.13 91.44 0)
-      (effects (font (size 1.27 1.27)) hide)
-    )
     (property "Quantity" "" (at 151.13 91.44 0)
       (effects (font (size 1.27 1.27)) hide)
@@
       (effects (font (size 1.27 1.27)) hide)
     )
+    (property "Farnell" "" (at 151.13 91.44 0)
+      (effects (font (size 1.27 1.27)) hide)
+    )
     (property "Field-1" "" (at 151.13 91.44 0)
       (effects (font (size 1.27 1.27)) hide)
@@
       (effects (font (size 1.27 1.27)) hide)
     )
-    (property "MANUFACTURER" "" (at 123.19 96.52 0)
-      (effects (font (size 1.27 1.27)) hide)
-    )
     (property "Quantity" "" (at 123.19 96.52 0)
       (effects (font (size 1.27 1.27)) hide)
     )
-    (property "Digikey" "" (at 123.19 96.52 0)
-      (effects (font (size 1.27 1.27)) hide)
-    )
-    (property "MPN" "" (at 123.19 96.52 0)
-      (effects (font (size 1.27 1.27)) hide)
-    )
-    (property "Mouser" "" (at 123.19 96.52 0)
+    (property "Digikey" "DS3231MZ+-ND" (at 123.19 96.52 0)
+      (effects (font (size 1.27 1.27)) hide)
+    )
+    (property "MPN" "DS3231MZ+" (at 123.19 96.52 0)
+      (effects (font (size 1.27 1.27)) hide)
+    )
+    (property "Mouser" "700-DS3231MZ+" (at 123.19 96.52 0)
+      (effects (font (size 1.27 1.27)) hide)
+    )
+    (property "Farnell" "" (at 123.19 96.52 0)
       (effects (font (size 1.27 1.27)) hide)
     )
     (property "Field-1" "" (at 123.19 96.52 0)
+      (effects (font (size 1.27 1.27)) hide)
+    )
+    (property "Manufacturer" "Maxim" (at 123.19 96.52 0)
       (effects (font (size 1.27 1.27)) hide)
     )
@@
       (effects (font (size 1.27 1.27)) hide)
     )
-    (property "MANUFACTURER" "" (at 93.98 77.47 0)
-      (effects (font (size 1.27 1.27)) hide)
-    )
     (property "Quantity" "" (at 93.98 77.47 0)
       (effects (font (size 1.27 1.27)) hide)
@@
       (effects (font (size 1.27 1.27)) hide)
     )
+    (property "Manufacturer" "Murata" (at 93.98 77.47 0)
+      (effects (font (size 1.27 1.27)) hide)
+    )
+    (property "Voltage" "50V" (at 93.98 77.47 0)
+      (effects (font (size 1.27 1.27)) hide)
+    )
+    (property "Farnell" "" (at 93.98 77.47 0)
+      (effects (font (size 1.27 1.27)) hide)
+    )
     (property "Field-1" "" (at 93.98 77.47 0)
       (effects (font (size 1.27 1.27)) hide)
     )
-    (property "Manufacturer" "Murata" (at 93.98 77.47 0)
-      (effects (font (size 1.27 1.27)) hide)
-    )
-    (property "Voltage" "50V" (at 93.98 77.47 0)
-      (effects (font (size 1.27 1.27)) hide)
-    )
