File: r5/src/_sdcard.kicad_sch (KiCad schematic)
At the start: 6 parts, among them J14 Micro_SD_Card_Det_JAE_ST11, U10 ESD7004, U11 ESD7004

Commit message: Oops, hadn't run the ERC for ages. Ran, passed. Add ERC and DRC exclusions where unavoidable
Parts:
- C29: MPN (none) -> GRM31CE70J476ME15L; Manufacturer (none) -> Murata; Mouser (none) -> 81-GRM31CE70J476ME5L
- J14: Digikey (none) -> 670-2695-6-ND; MPN (none) -> ST11S008V4HR2000; Manufacturer (none) -> JAE; Mouser (none) -> 656-ST11S008V4HR2000
- U10, U11: Digikey (none) -> ESD7004MUTAGOSDKR-ND; MPN (none) -> ESD7004MUTAG; Manufacturer (none) -> On Semi; Mouser (none) -> 863-ESD7004MUTAG
Changed lines of the file:
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@@
-      (effects (font (size 1.27 1.27)) hide)
-    )
-    (property "MANUFACTURER" "" (at 182.88 102.87 0)
       (effects (font (size 1.27 1.27)) hide)
     )
@@
       (effects (font (size 1.27 1.27)) hide)
     )
-    (property "Digikey" "" (at 182.88 102.87 0)
-      (effects (font (size 1.27 1.27)) hide)
-    )
-    (property "MPN" "" (at 182.88 102.87 0)
-      (effects (font (size 1.27 1.27)) hide)
-    )
-    (property "Mouser" "" (at 182.88 102.87 0)
+    (property "Digikey" "670-2695-6-ND" (at 182.88 102.87 0)
+      (effects (font (size 1.27 1.27)) hide)
+    )
+    (property "MPN" "ST11S008V4HR2000" (at 182.88 102.87 0)
+      (effects (font (size 1.27 1.27)) hide)
+    )
+    (property "Mouser" "656-ST11S008V4HR2000" (at 182.88 102.87 0)
+      (effects (font (size 1.27 1.27)) hide)
+    )
+    (property "Manufacturer" "JAE" (at 182.88 102.87 0)
+      (effects (font (size 1.27 1.27)) hide)
+    )
+    (property "Farnell" "" (at 182.88 102.87 0)
       (effects (font (size 1.27 1.27)) hide)
     )
@@
       (effects (font (size 1.27 1.27)) hide)
     )
-    (property "MANUFACTURER" "" (at 144.78 83.82 0)
-      (effects (font (size 1.27 1.27)) hide)
-    )
     (property "Quantity" "" (at 144.78 83.82 0)
       (effects (font (size 1.27 1.27)) hide)
@@
       (effects (font (size 1.27 1.27)) hide)
     )
+    (property "Farnell" "" (at 144.78 83.82 0)
+      (effects (font (size 1.27 1.27)) hide)
+    )
     (property "Field-1" "" (at 144.78 83.82 0)
       (effects (font (size 1.27 1.27)) hide)
@@
       (effects (font (size 1.27 1.27)) hide)
     )
-    (property "MANUFACTURER" "" (at 173.99 74.93 0)
-      (effects (font (size 1.27 1.27)) hide)
-    )
     (property "Quantity" "" (at 173.99 74.93 0)
       (effects (font (size 1.27 1.27)) hide)
@@
       (effects (font (size 1.27 1.27)) hide)
     )
+    (property "Manufacturer" "Murata" (at 173.99 74.93 0)
+      (effects (font (size 1.27 1.27)) hide)
+    )
+    (property "Voltage" "50V" (at 173.99 74.93 0)
+      (effects (font (size 1.27 1.27)) hide)
+    )
+    (property "Farnell" "" (at 173.99 74.93 0)
+      (effects (font (size 1.27 1.27)) hide)
+    )
     (property "Field-1" "" (at 173.99 74.93 0)
-      (effects (font (size 1.27 1.27)) hide)
-    )
-    (property "Manufacturer" "Murata" (at 173.99 74.93 0)
-      (effects (font (size 1.27 1.27)) hide)
-    )
-    (property "Voltage" "50V" (at 173.99 74.93 0)
       (effects (font (size 1.27 1.27)) hide)
     )
@@
       (effects (font (size 1.27 1.27)) hide)
     )
-    (property "MANUFACTURER" "" (at 162.56 74.93 0)
-      (effects (font (size 1.27 1.27)) hide)
-    )
     (property "Quantity" "" (at 162.56 74.93 0)
       (effects (font (size 1.27 1.27)) hide)
@@
       (effects (font (size 1.27 1.27)) hide)
     )
-    (property "MPN" "" (at 162.56 74.93 0)
-      (effects (font (size 1.27 1.27)) hide)
-    )
-    (property "Mouser" "" (at 162.56 74.93 0)
+    (property "MPN" "GRM31CE70J476ME15L " (at 162.56 74.93 0)
+      (effects (font (size 1.27 1.27)) hide)
+    )
+    (property "Mouser" "81-GRM31CE70J476ME5L " (at 162.56 74.93 0)
+      (effects (font (size 1.27 1.27)) hide)
+    )
+    (property "Manufacturer" "Murata" (at 162.56 74.93 0)
+      (effects (font (size 1.27 1.27)) hide)
+    )
+    (property "Farnell" "" (at 162.56 74.93 0)
       (effects (font (size 1.27 1.27)) hide)
     )
@@
       (effects (font (size 1.27 1.27)) hide)
     )
-    (property "MANUFACTURER" "" (at 118.11 123.19 0)
-      (effects (font (size 1.27 1.27)) hide)
-    )
     (property "Quantity" "" (at 118.11 123.19 0)
       (effects (font (size 1.27 1.27)) hide)
     )
-    (property "Digikey" "" (at 118.11 123.19 0)
-      (effects (font (size 1.27 1.27)) hide)
-    )
-    (property "MPN" "" (at 118.11 123.19 0)
-      (effects (font (size 1.27 1.27)) hide)
-    )
-    (property "Mouser" "" (at 118.11 123.19 0)
+    (property "Digikey" "ESD7004MUTAGOSDKR-ND" (at 118.11 123.19 0)
+      (effects (font (size 1.27 1.27)) hide)
+    )
+    (property "MPN" "ESD7004MUTAG" (at 118.11 123.19 0)
+      (effects (font (size 1.27 1.27)) hide)
+    )
+    (property "Mouser" "863-ESD7004MUTAG" (at 118.11 123.19 0)
+      (effects (font (size 1.27 1.27)) hide)
+    )
+    (property "Farnell" "" (at 118.11 123.19 0)
       (effects (font (size 1.27 1.27)) hide)
     )
     (property "Field-1" "" (at 118.11 123.19 0)
+      (effects (font (size 1.27 1.27)) hide)
+    )
+    (property "Manufacturer" "On Semi" (at 118.11 123.19 0)
       (effects (font (size 1.27 1.27)) hide)
     )
@@
       (effects (font (size 1.27 1.27)) hide)
     )
-    (property "MANUFACTURER" "" (at 135.89 123.19 0)
-      (effects (font (size 1.27 1.27)) hide)
-    )
     (property "Quantity" "" (at 135.89 123.19 0)
       (effects (font (size 1.27 1.27)) hide)
     )
-    (property "Digikey" "" (at 135.89 123.19 0)
-      (effects (font (size 1.27 1.27)) hide)
-    )
-    (property "MPN" "" (at 135.89 123.19 0)
-      (effects (font (size 1.27 1.27)) hide)
-    )
-    (property "Mouser" "" (at 135.89 123.19 0)
+    (property "Digikey" "ESD7004MUTAGOSDKR-ND" (at 135.89 123.19 0)
+      (effects (font (size 1.27 1.27)) hide)
+    )
+    (property "MPN" "ESD7004MUTAG" (at 135.89 123.19 0)
+      (effects (font (size 1.27 1.27)) hide)
+    )
+    (property "Mouser" "863-ESD7004MUTAG" (at 135.89 123.19 0)
+      (effects (font (size 1.27 1.27)) hide)
+    )
+    (property "Farnell" "" (at 135.89 123.19 0)
       (effects (font (size 1.27 1.27)) hide)
     )
@@
       (effects (font (size 1.27 1.27)) hide)
     )
+    (property "Manufacturer" "On Semi" (at 135.89 123.19 0)
+      (effects (font (size 1.27 1.27)) hide)
+    )
